Commit message: added urdf of the table

File: battery_cell_description/urdf/battery_cell.xacro (robot description, xacro)
@@ -39,4 +39,14 @@
       <child link="${nj_prefix}base_link"/>
   </joint>
+  <xacro:include filename="$(find battery_cell_description)/urdf/battery_table.xacro" />
+  <xacro:property name="table_prefix" value="'table_'" />
+  <xacro:battery_table prefix="${table_prefix}"/>
+  <joint name="world_to_table" type="fixed">
+      <origin
+        xyz="1 -1 0"
+        rpy="0 0 0" />
+      <parent link="world"/>
+      <child link="${table_prefix}base_link"/>
+  </joint>
   <gazebo>
     <plugin name="gazebo_ros_control" filename="libgazebo_ros_control.so">

Commit message: added urdf of the table and the omron mobile manipulator

File: battery_cell_description/urdf/battery_cell.xacro (robot description, xacro)
@@ -1,4 +1,14 @@
 <?xml version="1.0"?>
 <robot name="battery_cell" xmlns:xacro="http://www.ros.org/wiki/xacro">
+  <xacro:property name="M_PI" value="3.14159"/>
+  <xacro:property name="omron_x_pos_lower_limit" value="-2" />
+  <xacro:property name="omron_x_pos_upper_limit" value="5" />
+  <xacro:property name="omron_y_pos_lower_limit" value="-3" />
+  <xacro:property name="omron_y_pos_upper_limit" value="0.5" />
+  <xacro:property name="omron_rev_pos_lower_limit" value="${-M_PI}" />
+  <xacro:property name="omron_rev_pos_upper_limit" value="${M_PI}" />
+  <xacro:property name="omron_x_vel_limit" value="2" />
+  <xacro:property name="omron_y_vel_limit" value="2" />
+  <xacro:property name="omron_rev_vel_limit" value="${M_PI}" />
   <link name="world"/>
   <xacro:include filename="$(find kuka_structure_description)/urdf/kuka_structure.xacro" />
@@ -49,4 +59,47 @@
       <child link="${table_prefix}base_link"/>
   </joint>
+  <link name="omron_base_x"/>
+  <joint name="world_to_omron_base_x" type="prismatic">
+      <origin
+        xyz="0 0 0"
+        rpy="0 0 0" />
+      <parent link="world"/>
+      <child link="omron_base_x"/>
+      <axis
+        xyz="1 0 0" />
+      <limit lower="${omron_x_pos_lower_limit}" upper="${omron_x_pos_upper_limit}" effort="1000" velocity="${omron_x_vel_limit}"/>
+  </joint>
+  <link name="omron_base_y"/>
+  <joint name="omron_base_x_to_omron_base_y" type="prismatic">
+      <origin
+        xyz="0 0 0"
+        rpy="0 0 0" />
+      <parent link="omron_base_x"/>
+      <child link="omron_base_y"/>
+      <axis
+        xyz="0 1 0" />
+      <limit lower="${omron_y_pos_lower_limit}" upper="${omron_y_pos_upper_limit}" effort="1000" velocity="${omron_y_vel_limit}"/>
+  </joint>
+  <link name="omron_base_rev"/>
+  <joint name="omron_base_y_to_omron_base_rev" type="revolute">
+    <origin
+      xyz="0 0 0"
+      rpy="0 0 0" />
+    <parent link="omron_base_y"/>
+    <child link="omron_base_rev"/>
+    <axis
+      xyz="0 0 1" />
+    <limit lower="${omron_rev_pos_lower_limit}" upper="${omron_rev_pos_upper_limit}" effort="1000" velocity="${omron_rev_vel_limit}"/>
+  </joint>
+  <xacro:include filename="$(find mobile_manipulator_description)/urdf/mobile_manipulator.xacro" />
+  <xacro:property name="omron_prefix" value="'omron_'" />
+  <xacro:mobile_manipulator prefix="${omron_prefix}"/>
+  <joint name="omron_base_rev_to_omron_base_link" type="fixed">
+    <origin
+      xyz="0 0 0"
+      rpy="0 0 0" />
+    <parent link="omron_base_rev"/>
+    <child link="${omron_prefix}base_link"/>
+  </joint>
   <gazebo>
     <plugin name="gazebo_ros_control" filename="libgazebo_ros_control.so">

File: battery_cell_description/urdf/battery_table.xacro (robot description, xacro)
@@ -196,10 +196,10 @@
         value="${m_leg}" />
       <inertia
-        ixx="${1/12*m_table*(table_width*table_width + table_thickness*table_thickness)}"
+        ixx="${1/12*m_table*(table_length*table_length + table_thickness*table_thickness)}"
         ixy="0"
         ixz="0"
         iyy="${1/12*m_table*(table_width*table_width + table_thickness*table_thickness)}"
         iyz="0"
-        izz="${1/12*m_table*(table_width*table_width + table_width*table_width)}" />
+        izz="${1/12*m_table*(table_width*table_width + table_length*table_length)}" />
     </inertial>
     <visual>
@@ -208,10 +208,10 @@
         rpy="0 0 0" />
       <geometry>
-        <box size="${table_width} ${table_width} ${table_thickness}"/>
-      </geometry>
-      <material
-        name="">
-        <color
-          rgba="0.1176 0.5059 0.6902 1" />
+        <box size="${table_width} ${table_length} ${table_thickness}"/>
+      </geometry>
+      <material
+        name="">
+        <color
+          rgba="0.6608 0.6608 0.7878 1" />
       </material>
     </visual>
@@ -221,5 +221,5 @@
         rpy="0 0 0" />
       <geometry>
-        <box size="${table_width} ${table_width} ${table_thickness}"/>
+        <box size="${table_width} ${table_length} ${table_thickness}"/>
       </geometry>
     </collision>

Commit message: Revert "added urdf of the table and the omron mobile manipulator"
This reverts commit 0d1e508c9d791f1654b20868819d736ecd024839.

File: battery_cell_description/urdf/battery_cell.xacro (robot description, xacro)
@@ -1,14 +1,4 @@
 <?xml version="1.0"?>
 <robot name="battery_cell" xmlns:xacro="http://www.ros.org/wiki/xacro">
-  <xacro:property name="M_PI" value="3.14159"/>
-  <xacro:property name="omron_x_pos_lower_limit" value="-2" />
-  <xacro:property name="omron_x_pos_upper_limit" value="5" />
-  <xacro:property name="omron_y_pos_lower_limit" value="-3" />
-  <xacro:property name="omron_y_pos_upper_limit" value="0.5" />
-  <xacro:property name="omron_rev_pos_lower_limit" value="${-M_PI}" />
-  <xacro:property name="omron_rev_pos_upper_limit" value="${M_PI}" />
-  <xacro:property name="omron_x_vel_limit" value="2" />
-  <xacro:property name="omron_y_vel_limit" value="2" />
-  <xacro:property name="omron_rev_vel_limit" value="${M_PI}" />
   <link name="world"/>
   <xacro:include filename="$(find kuka_structure_description)/urdf/kuka_structure.xacro" />
@@ -59,47 +49,4 @@
       <child link="${table_prefix}base_link"/>
   </joint>
-  <link name="omron_base_x"/>
-  <joint name="world_to_omron_base_x" type="prismatic">
-      <origin
-        xyz="0 0 0"
-        rpy="0 0 0" />
-      <parent link="world"/>
-      <child link="omron_base_x"/>
-      <axis
-        xyz="1 0 0" />
-      <limit lower="${omron_x_pos_lower_limit}" upper="${omron_x_pos_upper_limit}" effort="1000" velocity="${omron_x_vel_limit}"/>
-  </joint>
-  <link name="omron_base_y"/>
-  <joint name="omron_base_x_to_omron_base_y" type="prismatic">
-      <origin
-        xyz="0 0 0"
-        rpy="0 0 0" />
-      <parent link="omron_base_x"/>
-      <child link="omron_base_y"/>
-      <axis
-        xyz="0 1 0" />
-      <limit lower="${omron_y_pos_lower_limit}" upper="${omron_y_pos_upper_limit}" effort="1000" velocity="${omron_y_vel_limit}"/>
-  </joint>
-  <link name="omron_base_rev"/>
-  <joint name="omron_base_y_to_omron_base_rev" type="revolute">
-    <origin
-      xyz="0 0 0"
-      rpy="0 0 0" />
-    <parent link="omron_base_y"/>
-    <child link="omron_base_rev"/>
-    <axis
-      xyz="0 0 1" />
-    <limit lower="${omron_rev_pos_lower_limit}" upper="${omron_rev_pos_upper_limit}" effort="1000" velocity="${omron_rev_vel_limit}"/>
-  </joint>
-  <xacro:include filename="$(find mobile_manipulator_description)/urdf/mobile_manipulator.xacro" />
-  <xacro:property name="omron_prefix" value="'omron_'" />
-  <xacro:mobile_manipulator prefix="${omron_prefix}"/>
-  <joint name="omron_base_rev_to_omron_base_link" type="fixed">
-    <origin
-      xyz="0 0 0"
-      rpy="0 0 0" />
-    <parent link="omron_base_rev"/>
-    <child link="${omron_prefix}base_link"/>
-  </joint>
   <gazebo>
     <plugin name="gazebo_ros_control" filename="libgazebo_ros_control.so">

File: battery_cell_description/urdf/battery_table.xacro (robot description, xacro)
@@ -196,10 +196,10 @@
         value="${m_leg}" />
       <inertia
-        ixx="${1/12*m_table*(table_length*table_length + table_thickness*table_thickness)}"
+        ixx="${1/12*m_table*(table_width*table_width + table_thickness*table_thickness)}"
         ixy="0"
         ixz="0"
         iyy="${1/12*m_table*(table_width*table_width + table_thickness*table_thickness)}"
         iyz="0"
-        izz="${1/12*m_table*(table_width*table_width + table_length*table_length)}" />
+        izz="${1/12*m_table*(table_width*table_width + table_width*table_width)}" />
     </inertial>
     <visual>
@@ -208,10 +208,10 @@
         rpy="0 0 0" />
       <geometry>
-        <box size="${table_width} ${table_length} ${table_thickness}"/>
-      </geometry>
-      <material
-        name="">
-        <color
-          rgba="0.6608 0.6608 0.7878 1" />
+        <box size="${table_width} ${table_width} ${table_thickness}"/>
+      </geometry>
+      <material
+        name="">
+        <color
+          rgba="0.1176 0.5059 0.6902 1" />
       </material>
     </visual>
@@ -221,5 +221,5 @@
         rpy="0 0 0" />
       <geometry>
-        <box size="${table_width} ${table_length} ${table_thickness}"/>
+        <box size="${table_width} ${table_width} ${table_thickness}"/>
       </geometry>
     </collision>

Commit message: fixed duplicate frames

File: battery_cell_description/urdf/battery_cell.xacro (robot description, xacro)
@@ -71,5 +71,5 @@
   </joint>
   <link name="omron_base_y"/>
-  <joint name="omron_base_x_to_omron_base_y" type="prismatic">
+  <joint name="omron_base_x_to_y" type="prismatic">
       <origin
         xyz="0 0 0"
@@ -81,24 +81,16 @@
       <limit lower="${omron_y_pos_lower_limit}" upper="${omron_y_pos_upper_limit}" effort="1000" velocity="${omron_y_vel_limit}"/>
   </joint>
-  <link name="omron_base_rev"/>
-  <joint name="omron_base_y_to_omron_base_rev" type="revolute">
+  <xacro:include filename="$(find mobile_manipulator_description)/urdf/mobile_manipulator.xacro" />
+  <xacro:property name="omron_prefix" value="'omron_'" />
+  <xacro:mobile_manipulator prefix="${omron_prefix}"/>
+  <joint name="omron_base_y_to_link" type="revolute">
     <origin
       xyz="0 0 0"
       rpy="0 0 0" />
     <parent link="omron_base_y"/>
-    <child link="omron_base_rev"/>
+    <child link="${omron_prefix}base_link"/>
     <axis
       xyz="0 0 1" />
     <limit lower="${omron_rev_pos_lower_limit}" upper="${omron_rev_pos_upper_limit}" effort="1000" velocity="${omron_rev_vel_limit}"/>
-  </joint>
-  <xacro:include filename="$(find mobile_manipulator_description)/urdf/mobile_manipulator.xacro" />
-  <xacro:property name="omron_prefix" value="'omron_'" />
-  <xacro:mobile_manipulator prefix="${omron_prefix}"/>
-  <joint name="omron_base_rev_to_omron_base_link" type="fixed">
-    <origin
-      xyz="0 0 0"
-      rpy="0 0 0" />
-    <parent link="omron_base_rev"/>
-    <child link="${omron_prefix}base_link"/>
   </joint>
   <gazebo>

File: battery_cell_description/urdf/battery_table.xacro (robot description, xacro)
@@ -49,5 +49,5 @@
     </collision>
   </link>
-  <joint name="${prefix}base_link_to_leg1" type="fixed">
+  <joint name="${prefix}base_to_leg1" type="fixed">
     <origin
       xyz="${table_width/2-leg_width/2} ${table_length/2-leg_width/2} 0"
@@ -93,5 +93,5 @@
     </collision>
   </link>
-  <joint name="${prefix}base_link_to_leg2" type="fixed">
+  <joint name="${prefix}base_to_leg2" type="fixed">
     <origin
       xyz="${table_width/2-leg_width/2} ${-table_length/2+leg_width/2} 0"
@@ -137,5 +137,5 @@
     </collision>
   </link>
-  <joint name="${prefix}base_link_to_leg3" type="fixed">
+  <joint name="${prefix}base_to_leg3" type="fixed">
     <origin
       xyz="${-table_width/2+leg_width/2} ${-table_length/2+leg_width/2} 0"
@@ -181,5 +181,5 @@
     </collision>
   </link>
-  <joint name="${prefix}base_link_to_leg4" type="fixed">
+  <joint name="${prefix}base_to_leg4" type="fixed">
     <origin
       xyz="${-table_width/2+leg_width/2} ${table_length/2-leg_width/2} 0"
@@ -225,5 +225,5 @@
     </collision>
   </link>
-  <joint name="${prefix}base_link_to_tabletop" type="fixed">
+  <joint name="${prefix}base_to_tabletop" type="fixed">
     <origin
       xyz="0 0 ${leg_height}"

Commit message: moved agv joints from cell to robot

File: battery_cell_description/urdf/battery_cell.xacro (robot description, xacro)
@@ -1,14 +1,4 @@
 <?xml version="1.0"?>
 <robot name="battery_cell" xmlns:xacro="http://www.ros.org/wiki/xacro">
-  <xacro:property name="M_PI" value="3.14159"/>
-  <xacro:property name="omron_x_pos_lower_limit" value="-2" />
-  <xacro:property name="omron_x_pos_upper_limit" value="5" />
-  <xacro:property name="omron_y_pos_lower_limit" value="-3" />
-  <xacro:property name="omron_y_pos_upper_limit" value="0.5" />
-  <xacro:property name="omron_rev_pos_lower_limit" value="${-M_PI}" />
-  <xacro:property name="omron_rev_pos_upper_limit" value="${M_PI}" />
-  <xacro:property name="omron_x_vel_limit" value="2" />
-  <xacro:property name="omron_y_vel_limit" value="2" />
-  <xacro:property name="omron_rev_vel_limit" value="${M_PI}" />
   <link name="world"/>
   <xacro:include filename="$(find kuka_structure_description)/urdf/kuka_structure.xacro" />
@@ -59,38 +49,13 @@
       <child link="${table_prefix}base_link"/>
   </joint>
-  <link name="omron_base_x"/>
-  <joint name="world_to_omron_base_x" type="prismatic">
-      <origin
-        xyz="0 0 0"
-        rpy="0 0 0" />
-      <parent link="world"/>
-      <child link="omron_base_x"/>
-      <axis
-        xyz="1 0 0" />
-      <limit lower="${omron_x_pos_lower_limit}" upper="${omron_x_pos_upper_limit}" effort="1000" velocity="${omron_x_vel_limit}"/>
-  </joint>
-  <link name="omron_base_y"/>
-  <joint name="omron_base_x_to_y" type="prismatic">
-      <origin
-        xyz="0 0 0"
-        rpy="0 0 0" />
-      <parent link="omron_base_x"/>
-      <child link="omron_base_y"/>
-      <axis
-        xyz="0 1 0" />
-      <limit lower="${omron_y_pos_lower_limit}" upper="${omron_y_pos_upper_limit}" effort="1000" velocity="${omron_y_vel_limit}"/>
-  </joint>
   <xacro:include filename="$(find mobile_manipulator_description)/urdf/mobile_manipulator.xacro" />
   <xacro:property name="omron_prefix" value="'omron_'" />
   <xacro:mobile_manipulator prefix="${omron_prefix}"/>
-  <joint name="omron_base_y_to_link" type="revolute">
+  <joint name="world_to_omron" type="fixed">
     <origin
-      xyz="0 0 0"
+      xyz="4.5 -3 0"
       rpy="0 0 0" />
-    <parent link="omron_base_y"/>
+    <parent link="world"/>
     <child link="${omron_prefix}base_link"/>
-    <axis
-      xyz="0 0 1" />
-    <limit lower="${omron_rev_pos_lower_limit}" upper="${omron_rev_pos_upper_limit}" effort="1000" velocity="${omron_rev_vel_limit}"/>
   </joint>
   <gazebo>
