Commit message: workin

File: battery_cell_description/urdf/battery_cell_ros2_control.xacro (robot description, xacro)
@@ -1,2 +1,30 @@
+NON E' USATO DA NESSUNA PARTE
+NON E' USATO DA NESSUNA PARTE
+NON E' USATO DA NESSUNA PARTE
+NON E' USATO DA NESSUNA PARTE
+NON E' USATO DA NESSUNA PARTE
+NON E' USATO DA NESSUNA PARTE
+NON E' USATO DA NESSUNA PARTE
+NON E' USATO DA NESSUNA PARTE
+NON E' USATO DA NESSUNA PARTE
+NON E' USATO DA NESSUNA PARTE
+NON E' USATO DA NESSUNA PARTE
+NON E' USATO DA NESSUNA PARTE
+NON E' USATO DA NESSUNA PARTE
+NON E' USATO DA NESSUNA PARTE
+NON E' USATO DA NESSUNA PARTE
+NON E' USATO DA NESSUNA PARTE
+NON E' USATO DA NESSUNA PARTE
+NON E' USATO DA NESSUNA PARTE
+NON E' USATO DA NESSUNA PARTE
+NON E' USATO DA NESSUNA PARTE
+NON E' USATO DA NESSUNA PARTE
+NON E' USATO DA NESSUNA PARTE
+NON E' USATO DA NESSUNA PARTE
+NON E' USATO DA NESSUNA PARTE
+NON E' USATO DA NESSUNA PARTE
+NON E' USATO DA NESSUNA PARTE
+NON E' USATO DA NESSUNA PARTE
+NON E' USATO DA NESSUNA PARTE
 <?xml version="1.0"?>
 <robot xmlns:xacro="http://www.ros.org/wiki/xacro">
@@ -41,7 +69,7 @@
         <command_interface name="d_output.3"/>
         <command_interface name="d_output.4"/>
-        <command_interface name="d_output.5"/>
+        <command_interface name="screwdriver_lp"/>
         <command_interface name="d_output.6"/>
-        <command_interface name="d_output.7"/>
+        <command_interface name="screwdriver_hp"/>
         <ec_module name="EL2008">
           <plugin>ethercat_generic_plugins/GenericEcSlave</plugin>

File: battery_cell_description/urdf/battery_cell_rviz.xacro (robot description, xacro)
@@ -2,9 +2,14 @@
 <robot name="battery_cell" xmlns:xacro="http://www.ros.org/wiki/xacro">
   <xacro:arg name="use_fake_hardware" default="true"/>
+  <xacro:arg name="use_kuka_fake_hardware" default="true"/>
+  <xacro:arg name="use_linear_axis_fake_hardware" default="true"/>
+  <xacro:arg name="use_comau_fake_hardware" default="true"/>
   <xacro:arg name="include_omron" default="true"/>
   <xacro:property name="use_fake_hardware" value="'$(arg use_fake_hardware)'" />
+  <!-- <xacro:property name="use_kuka_fake_hardware" value="'$(arg use_kuka_fake_hardware)'" /> -->
   <link name="world"/>
   <xacro:include filename="$(find battery_cell_description)/urdf/kuka_setup.xacro" />
-  <xacro:kuka_setup use_fake_hardware="${use_fake_hardware}"/>
+  <xacro:kuka_setup use_kuka_fake_hardware="$(arg use_kuka_fake_hardware)"
+                    use_linear_axis_fake_hardware="$(arg use_linear_axis_fake_hardware)"/>
   <joint name="world_to_kuka" type="fixed">
       <origin
@@ -25,5 +30,6 @@
   </joint>
   <xacro:include filename="$(find battery_cell_description)/urdf/comau_setup.xacro" />
-  <xacro:comau_setup use_fake_hardware="${use_fake_hardware}"/>
+  <!-- <xacro:comau_setup use_fake_hardware="${use_fake_hardware}"/> -->
+  <xacro:comau_setup use_fake_hardware="$(arg use_comau_fake_hardware)"/>
   <joint name="world_to_comau" type="fixed">
       <origin
@@ -43,3 +49,246 @@
     </joint>
   </xacro:if>
+  <!-- increased collisions -->
+  <!-- FLOOR -->
+  <xacro:property name="floor_thickness" value="0.10" />
+  <xacro:property name="floor_length" value="${8.20+2*floor_thickness}" />
+  <xacro:property name="floor_width" value="11.0" />
+  <link name="floor_link">
+    <inertial>
+      <origin
+        xyz="0 0 ${floor_thickness/2}"
+        rpy="0 0 0" />
+      <mass
+        value="0" />
+      <inertia
+        ixx="0"
+        ixy="0"
+        ixz="0"
+        iyy="0"
+        iyz="0"
+        izz="0" />
+    </inertial>
+    <visual>
+      <origin
+        xyz="0 0 ${floor_thickness/2}"
+        rpy="0 0 0" />
+      <geometry>
+        <box size="${floor_width} ${floor_length} ${floor_thickness}"/>
+      </geometry>
+      <material
+        name="">
+        <color
+          rgba="0.6608 0.6608 0.7878 1" />
+      </material>
+    </visual>
+    <collision>
+      <origin
+        xyz="0 0 ${floor_thickness/2}"
+        rpy="0 0 0" />
+      <geometry>
+        <box size="${floor_width} ${floor_length} ${floor_thickness}"/>
+      </geometry>
+    </collision>
+  </link>
+  <joint name="world_to_floor" type="fixed">
+    <origin
+      xyz="0.5 -1.5 ${-floor_thickness}"
+      rpy="0 0 0" />
+    <parent link="world"/>
+    <child link="floor_link"/>
+  </joint>
+  <!-- REAR WALL -->
+  <xacro:property name="wall_thickness" value="0.10" />
+  <xacro:property name="wall_height" value="4.0" />
+  <xacro:property name="wall_width" value="11.0" />
+  <link name="wall_link">
+    <inertial>
+      <origin
+        xyz="0.0 0.0 ${-wall_thickness/2}"
+        rpy="0.0 0.0 0.0" />
+      <mass
+        value="0" />
+      <inertia
+        ixx="0"
+        ixy="0"
+        ixz="0"
+        iyy="0"
+        iyz="0"
+        izz="0" />
+    </inertial>
+    <visual>
+      <origin
+        xyz="0.0 0.0 ${-wall_thickness/2}"
+        rpy="0.0 0.0 0.0" />
+      <geometry>
+        <box size="${wall_height} ${wall_width} ${wall_thickness}"/>
+      </geometry>
+      <material
+        name="">
+        <color
+          rgba="0.6608 0.6608 0.7878 1" />
+      </material>
+    </visual>
+    <collision>
+      <origin
+        xyz="0.0 0.0 ${-wall_thickness/2}"
+        rpy="0.0 0.0 0.0" />
+      <geometry>
+        <box size="${wall_height} ${wall_width} ${wall_thickness}"/>
+      </geometry>
+    </collision>
+  </link>
+  <joint name="world_to_wall" type="fixed">
+    <origin
+      xyz="0.5 2.60 ${wall_height/2}"
+      rpy="1.5708 1.5708 0" />
+    <parent link="world"/>
+    <child link="wall_link"/>
+  </joint>
+  <!-- HORIZONTAL WALL-MOUNTED SUPPORT -->
+  <xacro:property name="support_height" value="1.20" />
+  <xacro:property name="support_length" value="0.50" />
+  <xacro:property name="support_width" value="${wall_width}" />
+  <xacro:property name="support_vert_offset" value="${wall_height/2-2.45}" />
+  <link name="support_link">
+    <inertial>
+      <origin
+        xyz="0.0 0.0 ${-support_height/2}"
+        rpy="0.0 0.0 0.0" />
+      <mass
+        value="0" />
+      <inertia
+        ixx="0"
+        ixy="0"
+        ixz="0"
+        iyy="0"
+        iyz="0"
+        izz="0" />
+    </inertial>
+    <visual>
+      <origin
+        xyz="0.0 0.0 ${-support_height/2}"
+        rpy="0.0 0.0 0.0" />
+      <geometry>
+        <box size="${support_length} ${support_width} ${support_height}"/>
+      </geometry>
+      <material
+        name="">
+        <color
+          rgba="0.1176 0.5059 0.6902 0.5" />
+      </material>
+    </visual>
+    <collision>
+      <origin
+        xyz="0.0 0.0 ${-support_height/2}"
+        rpy="0.0 0.0 0.0" />
+      <geometry>
+        <box size="${support_length} ${support_width} ${support_height}"/>
+      </geometry>
+    </collision>
+  </link>
+  <joint name="wall_to_support" type="fixed">
+    <origin
+      xyz="${support_vert_offset} 0.0 ${support_height}"
+      rpy="0.0 0.0 0.0" />
+    <parent link="wall_link"/>
+    <child link="support_link"/>
+  </joint>
+  <!-- REAL WALL INCREASED -->
+  <xacro:property name="wall_fake_height" value="${wall_height}" />
+  <xacro:property name="wall_fake_length" value="0.50" />
+  <xacro:property name="wall_fake_width" value="${wall_width}" />
+  <link name="wall_fake_link">
+    <inertial>
+      <origin
+        xyz="0.0 0.0 ${-wall_fake_height/2}"
+        rpy="0.0 0.0 0.0" />
+      <mass
+        value="0" />
+      <inertia
+        ixx="0"
+        ixy="0"
+        ixz="0"
+        iyy="0"
+        iyz="0"
+        izz="0" />
+    </inertial>
+    <visual>
+      <origin
+        xyz="0.0 0.0 ${-wall_fake_height/2}"
+        rpy="0.0 0.0 0.0" />
+      <geometry>
+        <box size="${wall_fake_length} ${wall_fake_width} ${wall_fake_height}"/>
+      </geometry>
+      <material
+        name="">
+        <color
+          rgba="0.1176 0.5059 0.6902 0.5" />
+      </material>
+    </visual>
+    <collision>
+      <origin
+        xyz="0.0 0.0 ${-wall_fake_height/2}"
+        rpy="0.0 0.0 0.0" />
+      <geometry>
+        <box size="${wall_fake_length} ${wall_fake_width} ${wall_fake_height}"/>
+      </geometry>
+    </collision>
+  </link>
+  <joint name="wall_to_wall_fake" type="fixed">
+    <origin
+      xyz="${wall_height/2} 0.0 ${wall_fake_length/2}"
+      rpy="0.0 1.5708 0.0" />
+    <parent link="wall_link"/>
+    <child link="wall_fake_link"/>
+  </joint>
+  <!-- KUKA CONTROLLER BOX -->
+  <xacro:property name="kuka_controller_height" value="1.40" /> <!-- TODO -->
+  <xacro:property name="kuka_controller_length" value="1.20" /> <!-- TODO -->
+  <xacro:property name="kuka_controller_width" value="1.20" />  <!-- TODO -->
+  <link name="kuka_controller_link">
+    <inertial>
+      <origin
+        xyz="0.0 0.0 0.0"
+        rpy="0.0 0.0 0.0" />
+      <mass
+        value="0" />
+      <inertia
+        ixx="0"
+        ixy="0"
+        ixz="0"
+        iyy="0"
+        iyz="0"
+        izz="0" />
+    </inertial>
+    <visual>
+      <origin
+        xyz="0.0 0.0 0.0"
+        rpy="0.0 0.0 0.0" />
+      <geometry>
+        <box size="${kuka_controller_length} ${kuka_controller_width} ${kuka_controller_height}"/>
+      </geometry>
+      <material
+        name="">
+        <color
+          rgba="0.1176 0.5059 0.6902 0.5" />
+      </material>
+    </visual>
+    <collision>
+      <origin
+        xyz="0.0 0.0 0.0"
+        rpy="0.0 0.0 0.0" />
+      <geometry>
+        <box size="${kuka_controller_length} ${kuka_controller_width} ${kuka_controller_height}"/>
+      </geometry>
+    </collision>
+  </link>
+  <joint name="structure_to_kuka_controller" type="fixed">
+    <origin
+      xyz="-3.0 1.0 0.0"
+      rpy="0.0 0.0 0.0" />    <!-- TODO -->
+    <parent link="structure_base_link"/>
+    <child link="kuka_controller_link"/>
+  </joint>
+  <!-- end increased collisions -->
 </robot>

File: battery_cell_description/urdf/kuka_setup.xacro (robot description, xacro)
@@ -1,5 +1,8 @@
 <?xml version="1.0"?>
 <robot xmlns:xacro="http://www.ros.org/wiki/xacro">
-  <xacro:macro name="kuka_setup"  params="prefix:='' robot_name:='kuka' use_fake_hardware='false'">
+  <xacro:macro name="kuka_setup"  params="prefix:=''
+                                          robot_name:='kuka'
+                                          use_kuka_fake_hardware='false'
+                                          use_linear_axis_fake_hardware='false'">
     <xacro:include filename="$(find kuka_structure_description)/urdf/kuka_structure.xacro" />
     <xacro:property name="kuka_structure_prefix" value="'structure_'" />
@@ -7,5 +10,5 @@
     <xacro:kuka_structure prefix="${prefix}${kuka_structure_prefix}"
                           name="${prefix}${kuka_structure_name}"
-                          use_fake_hardware="${use_fake_hardware}"/>
+                          use_fake_hardware="${use_linear_axis_fake_hardware}"/>
     <xacro:include filename="$(find kr_50_r2500_description)/urdf/kr_50_r2500.xacro" />
     <xacro:property name="kuka_prefix" value="'kuka_'" />
@@ -13,5 +16,5 @@
     <xacro:kr_50_r2500 prefix="${prefix}${kuka_prefix}"
                        name="${prefix}${kuka_name}"
-                       use_fake_hardware="${use_fake_hardware}" />
+                       use_fake_hardware="${use_kuka_fake_hardware}" />
     <joint name="kuka_structure_to_kr_50_r2500" type="fixed">
         <origin
@@ -152,9 +155,14 @@
 <!-- increased collisions -->
     <xacro:property name="fake_foot_lenght_x" value="0.87" />
-    <xacro:property name="fake_foot_lenght_y" value="1.5" />
-    <xacro:property name="fake_foot_lenght_z" value="1.3" />
-    <xacro:property name="fake_structure_lenght_x" value="4.3" />
-    <xacro:property name="fake_structure_lenght_y" value="1.5" />
-    <xacro:property name="fake_structure_lenght_z" value="4.0" />
+    <xacro:property name="fake_foot_lenght_y" value="1.50" />
+    <xacro:property name="fake_foot_lenght_z" value="1.30" />
+    <xacro:property name="fake_pillar_lenght_x" value="0.60" />
+    <xacro:property name="fake_pillar_lenght_y" value="0.70" />
+    <xacro:property name="fake_pillar_lenght_z" value="2.80" />
+    <xacro:property name="fake_structure_lenght_x" value="4.30" />
+    <xacro:property name="fake_structure_lenght_y" value="1.50" />
+    <xacro:property name="fake_structure_lenght_z" value="2.00" />
+    <xacro:property name="fake_structure_offset_z" value="2.50" />
+    <!-- RIGHT FOOT -->
     <joint name="${prefix}${kuka_prefix}fake_structure_right_foot" type="fixed">
       <origin
@@ -198,4 +206,47 @@
       </collision>
     </link>
+    <!-- RIGHT PILLAR -->
+    <joint name="${prefix}${kuka_prefix}fake_structure_right_pillar" type="fixed">
+      <origin
+        xyz="0.10 0.50 0"
+        rpy="0 0 0" />
+      <parent link="${prefix}${kuka_structure_prefix}base_link"/>
+      <child link="${prefix}${kuka_structure_prefix}fake_structure_right_pillar"/>
+    </joint>
+    <link name="${prefix}${kuka_structure_prefix}fake_structure_right_pillar">
+      <inertial>
+        <origin xyz="0 0 00" rpy="0 0 0" />
+        <mass value="10000" />
+        <inertia
+          ixx="0.1"
+          ixy="0.0"
+          ixz="0.0"
+          iyy="0.1"
+          iyz="0.0"
+          izz="0.1" />
+      </inertial>
+      <visual>
+        <origin
+          xyz="${fake_pillar_lenght_x/2} ${fake_pillar_lenght_y/2} ${fake_pillar_lenght_z/2}"
+          rpy="0 0 0" />
+        <geometry>
+          <box size="${fake_pillar_lenght_x} ${fake_pillar_lenght_y} ${fake_pillar_lenght_z}"/>
+        </geometry>
+        <material
+          name="">
+          <color
+            rgba="0.1176 0.5059 0.6902 0.5" />
+        </material>
+      </visual>
+      <collision>
+        <origin
+          xyz="${fake_pillar_lenght_x/2} ${fake_pillar_lenght_y/2} ${fake_pillar_lenght_z/2}"
+          rpy="0 0 0" />
+        <geometry>
+          <box size="${fake_pillar_lenght_x} ${fake_pillar_lenght_y} ${fake_pillar_lenght_z}"/>
+        </geometry>
+      </collision>
+    </link>
+    <!-- LEFT FOOT -->
     <joint name="${prefix}${kuka_prefix}fake_structure_left_foot" type="fixed">
       <origin
@@ -239,7 +290,50 @@
       </collision>
     </link>
+    <!-- LEFT PILLAR -->
+    <joint name="${prefix}${kuka_prefix}fake_structure_left_pillar" type="fixed">
+      <origin
+        xyz="2.55 0.50 0"
+        rpy="0 0 0" />
+      <parent link="${prefix}${kuka_structure_prefix}base_link"/>
+      <child link="${prefix}${kuka_structure_prefix}fake_structure_left_pillar"/>
+    </joint>
+    <link name="${prefix}${kuka_structure_prefix}fake_structure_left_pillar">
+      <inertial>
+        <origin xyz="0 0 00" rpy="0 0 0" />
+        <mass value="10000" />
+        <inertia
+          ixx="0.1"
+          ixy="0.0"
+          ixz="0.0"
+          iyy="0.1"
+          iyz="0.0"
+          izz="0.1" />
+      </inertial>
+      <visual>
+        <origin
+          xyz="${fake_pillar_lenght_x/2} ${fake_pillar_lenght_y/2} ${fake_pillar_lenght_z/2}"
+          rpy="0 0 0" />
+        <geometry>
+          <box size="${fake_pillar_lenght_x} ${fake_pillar_lenght_y} ${fake_pillar_lenght_z}"/>
+        </geometry>
+        <material
+          name="">
+          <color
+            rgba="0.1176 0.5059 0.6902 0.5" />
+        </material>
+      </visual>
+      <collision>
+        <origin
+          xyz="${fake_pillar_lenght_x/2} ${fake_pillar_lenght_y/2} ${fake_pillar_lenght_z/2}"
+          rpy="0 0 0" />
+        <geometry>
+          <box size="${fake_pillar_lenght_x} ${fake_pillar_lenght_y} ${fake_pillar_lenght_z}"/>
+        </geometry>
+      </collision>
+    </link>
+    <!-- PORTAL STRUCTURE -->
     <joint name="${prefix}${kuka_prefix}fake_structure" type="fixed">
       <origin
-        xyz="-0.45 0.2  0"
+        xyz="-0.45 0.2  ${fake_structure_offset_z}"
         rpy="0 0 0" />
       <parent link="${prefix}${kuka_structure_prefix}base_link"/>
