Commit message: trjs

File: battery_cell_description/urdf/battery_cell_GPIO_ros2_control.xacro (robot description, xacro)
@@ -1,34 +1,21 @@
-NON E' USATO DA NESSUNA PARTE
-NON E' USATO DA NESSUNA PARTE
-NON E' USATO DA NESSUNA PARTE
-NON E' USATO DA NESSUNA PARTE
-NON E' USATO DA NESSUNA PARTE
-NON E' USATO DA NESSUNA PARTE
-NON E' USATO DA NESSUNA PARTE
-NON E' USATO DA NESSUNA PARTE
-NON E' USATO DA NESSUNA PARTE
-NON E' USATO DA NESSUNA PARTE
-NON E' USATO DA NESSUNA PARTE
-NON E' USATO DA NESSUNA PARTE
-NON E' USATO DA NESSUNA PARTE
-NON E' USATO DA NESSUNA PARTE
-NON E' USATO DA NESSUNA PARTE
-NON E' USATO DA NESSUNA PARTE
-NON E' USATO DA NESSUNA PARTE
-NON E' USATO DA NESSUNA PARTE
-NON E' USATO DA NESSUNA PARTE
-NON E' USATO DA NESSUNA PARTE
-NON E' USATO DA NESSUNA PARTE
-NON E' USATO DA NESSUNA PARTE
-NON E' USATO DA NESSUNA PARTE
-NON E' USATO DA NESSUNA PARTE
-NON E' USATO DA NESSUNA PARTE
-NON E' USATO DA NESSUNA PARTE
-NON E' USATO DA NESSUNA PARTE
-NON E' USATO DA NESSUNA PARTE
 <?xml version="1.0"?>
 <robot xmlns:xacro="http://www.ros.org/wiki/xacro">
-  <xacro:macro name="battery_cell_ros2_control" >
-    <ros2_control name="kuka_structure" type="system">
+  <!-- <xacro:macro name="battery_cell_GPIO_ros2_control" params="name:='battery_cell_GPIO'
+                                                             master_id:=0
+                                                             use_fake_hardware:=true"> -->
+  <xacro:macro name="battery_cell_GPIO_ros2_control" params="name:='battery_cell_GPIO'">
+    <!-- <ros2_control name="${name}" type="system"> -->
+      <!-- <hardware>
+        <xacro:if value="${use_fake_hardware}">
+          <plugin>mock_components/GenericSystem</plugin>
+          <param name="mock_sensor_commands">false</param>
+          <param name="state_following_offset">0.0</param>
+        </xacro:if>
+        <xacro:unless value="${use_fake_hardware}">
+          <plugin>ethercat_driver/EthercatDriver</plugin>
+          <param name="master_id">${master_id}</param>
+          <param name="control_frequency">1000</param>
+        </xacro:unless>
+      </hardware> -->
       <gpio name="digital_inputs">
         <state_interface name="lubrication_state"/>
@@ -44,5 +31,5 @@
           <param name="alias">0</param>
           <param name="position">2</param>
-          <param name="slave_config">$(find kuka_structure_description)/config/EL1008_ethercat_config.yaml</param>
+          <param name="slave_config">$(find battery_cell_description)/config/ethercat/EL1008_ethercat_config.yaml</param>
         </ec_module>
       </gpio>
@@ -50,5 +37,5 @@
         <command_interface name="lubrication_command"/>
         <command_interface name="d_output.1"/>
-        <command_interface name="pneumatic_gripper"/>
+        <command_interface name="kuka_tool_change"/> <!-- TRUE to open, FALSE to close -->
         <command_interface name="d_output.3"/>
         <command_interface name="d_output.4"/>
@@ -60,5 +47,5 @@
           <param name="alias">0</param>
           <param name="position">3</param>
-          <param name="slave_config">$(find kuka_structure_description)/config/EL2008_ethercat_config_1.yaml</param>
+          <param name="slave_config">$(find battery_cell_description)/config/ethercat/EL2008_ethercat_config_1.yaml</param>
         </ec_module>
       </gpio>
@@ -76,5 +63,5 @@
           <param name="alias">0</param>
           <param name="position">4</param>
-          <param name="slave_config">$(find kuka_structure_description)/config/EL2008_ethercat_config_2.yaml</param>
+          <param name="slave_config">$(find battery_cell_description)/config/ethercat/EL2008_ethercat_config_2.yaml</param>
         </ec_module>
       </gpio>
@@ -99,9 +86,9 @@
           <param name="alias">0</param>
           <param name="position">5</param>
-          <param name="slave_config">$(find kuka_structure_description)/config/EL3008_ethercat_config.yaml</param>
-          <param name="sensor_runtime_matrix">$(find kuka_structure_description)/config/ati_sensor_runtime_matrix.yaml</param>
+          <param name="slave_config">$(find battery_cell_description)/config/ethercat/EL3008_ethercat_config.yaml</param>
+          <param name="sensor_runtime_matrix">$(find battery_cell_description)/config/ethercat/ati_sensor_runtime_matrix.yaml</param>
         </ec_module>
       </gpio>
-    </ros2_control>
+    <!-- </ros2_control> -->
   </xacro:macro>
 </robot>

File: battery_cell_description/urdf/battery_cell_rviz.xacro (robot description, xacro)
@@ -3,6 +3,7 @@
   <xacro:arg name="use_fake_hardware" default="true"/>
   <xacro:arg name="use_kuka_fake_hardware" default="true"/>
-  <xacro:arg name="use_linear_axis_fake_hardware" default="true"/>
+  <!-- <xacro:arg name="use_linear_axis_fake_hardware" default="true"/> -->
   <xacro:arg name="use_comau_fake_hardware" default="true"/>
+  <xacro:arg name="use_ethercat_fake_hardware" default="true"/>
   <xacro:arg name="include_omron" default="true"/>
   <xacro:property name="use_fake_hardware" value="'$(arg use_fake_hardware)'" />
@@ -11,5 +12,8 @@
   <xacro:include filename="$(find battery_cell_description)/urdf/kuka_setup.xacro" />
   <xacro:kuka_setup use_kuka_fake_hardware="$(arg use_kuka_fake_hardware)"
-                    use_linear_axis_fake_hardware="$(arg use_linear_axis_fake_hardware)"/>
+                    use_linear_axis_fake_hardware="$(arg use_ethercat_fake_hardware)"/>
+  <!-- Include ROS2 HW interface definitions for GPIO modules -->
+  <xacro:include filename="$(find battery_cell_description)/urdf/ethercat_ros2_control.xacro"/>
+  <xacro:ethercat_ros2_control use_fake_hardware="$(arg use_ethercat_fake_hardware)"/>
   <joint name="world_to_kuka" type="fixed">
       <origin
@@ -49,4 +53,6 @@
     </joint>
   </xacro:if>
+  <!-- <xacro:include filename="$(find battery_cell_description)/urdf/battery_cell_GPIO_ros2_control.xacro" />
+  <xacro:battery_cell_GPIO_ros2_control use_fake_hardware="$(arg use_GPIO_fake_hardware)"/> -->
   <!-- increased collisions -->
   <!-- FLOOR -->

File: battery_cell_description/urdf/kuka_setup.xacro (robot description, xacro)
@@ -10,5 +10,6 @@
     <xacro:kuka_structure prefix="${prefix}${kuka_structure_prefix}"
                           name="${prefix}${kuka_structure_name}"
-                          use_fake_hardware="${use_linear_axis_fake_hardware}"/>
+                          use_fake_hardware="${use_linear_axis_fake_hardware}"
+                          external_ethercat_ros2_control="true"/>
     <xacro:include filename="$(find kr_50_r2500_description)/urdf/kr_50_r2500.xacro" />
     <xacro:property name="kuka_prefix" value="'kuka_'" />
