Commit message: bridge configuration updated

File: battery_cell_description/urdf/battery_cell_rviz.xacro (robot description, xacro)
@@ -23,5 +23,5 @@
     <child link="${table_prefix}base_link"/>
   </joint>
- <xacro:include filename="$(find battery_cell_description)/urdf/comau_setup.xacro" />
+ <!-- <xacro:include filename="$(find battery_cell_description)/urdf/comau_setup.xacro" />
   <xacro:comau_setup use_fake_hardware="${use_fake_hardware}"/>
   <joint name="world_to_comau" type="fixed">
@@ -31,4 +31,4 @@
       <parent link="world"/>
       <child link="comau_basement"/>
-  </joint>
+  </joint> -->
 </robot>

Commit message: wip: new moveit_config; omron; launcher

File: battery_cell_description/urdf/battery_cell_rviz.xacro (robot description, xacro)
@@ -18,17 +18,25 @@
   <joint name="world_to_table" type="fixed">
     <origin
-      xyz="-0.30 -1.58 0"
+      xyz="0.025 -1.58 0"
       rpy="0 0 0" />
     <parent link="world"/>
     <child link="${table_prefix}base_link"/>
   </joint>
- <!-- <xacro:include filename="$(find battery_cell_description)/urdf/comau_setup.xacro" />
-  <xacro:comau_setup use_fake_hardware="${use_fake_hardware}"/>
+  <xacro:include filename="$(find battery_cell_description)/urdf/comau_setup.xacro" />
+  <xacro:comau_setup use_fake_hardware="true"/>
+  <!-- <xacro:comau_setup use_fake_hardware="${use_fake_hardware}"/> -->
   <joint name="world_to_comau" type="fixed">
       <origin
         xyz="-2.708 -0.430 0"
-        rpy="0 0 3.14159" />
+        rpy="0 0 0" />
       <parent link="world"/>
       <child link="comau_basement"/>
-  </joint> -->
+  </joint>
+  <xacro:include filename="$(find battery_cell_description)/urdf/omron_setup.xacro" />
+  <xacro:omron_setup use_fake_hardware="${use_fake_hardware}"/>
+  <joint name="world_to_map" type="fixed">
+    <parent link="world"/>
+    <child link="omron/map"/>
+    <origin xyz="0.0 -4.0 0.0"/>
+  </joint>
 </robot>

File: battery_cell_description/urdf/comau_setup.xacro (robot description, xacro)
@@ -40,6 +40,7 @@
       </collision>
     </link>
-    <xacro:include filename="$(find nj_220_2_7_description)/urdf/nj_220_2_7.xacro" />
-    <xacro:nj_220_2_7 prefix="${prefix}${nj_prefix}"/>
+    <xacro:include filename="$(find nj-220-27_description)/urdf/nj-220-27.xacro" />
+    <xacro:nj-220-27 prefix="${prefix}${nj_prefix}"
+                     use_fake_hardware="${use_fake_hardware}"/>
     <joint name="${prefix}${nj_prefix}basement_to_robot" type="fixed">
       <origin
@@ -50,5 +51,5 @@
     </joint>
   <!-- increased collisions -->
-    <xacro:property name="fake_robot_lenght_x" value="4" />
+    <!-- <xacro:property name="fake_robot_lenght_x" value="4" />
     <xacro:property name="fake_robot_lenght_y" value="3" />
     <xacro:property name="fake_robot_lenght_z" value="3" />
@@ -93,5 +94,5 @@
         </geometry>
       </collision>
-    </link>
+    </link> -->
   <!-- end increased collisions -->
   </xacro:macro>

File: battery_cell_moveit_config/config/battery_cell.ros2_control.xacro (robot description, xacro)
@@ -99,4 +99,46 @@
                 <state_interface name="velocity"/>
             </joint>
+            <joint name="omron/joint_1">
+                <command_interface name="position"/>
+                <state_interface name="position">
+                  <param name="initial_value">${initial_positions['omron/joint_1']}</param>
+                </state_interface>
+                <state_interface name="velocity"/>
+            </joint>
+            <joint name="omron/joint_2">
+                <command_interface name="position"/>
+                <state_interface name="position">
+                  <param name="initial_value">${initial_positions['omron/joint_2']}</param>
+                </state_interface>
+                <state_interface name="velocity"/>
+            </joint>
+            <joint name="omron/joint_3">
+                <command_interface name="position"/>
+                <state_interface name="position">
+                  <param name="initial_value">${initial_positions['omron/joint_3']}</param>
+                </state_interface>
+                <state_interface name="velocity"/>
+            </joint>
+            <joint name="omron/joint_4">
+                <command_interface name="position"/>
+                <state_interface name="position">
+                  <param name="initial_value">${initial_positions['omron/joint_4']}</param>
+                </state_interface>
+                <state_interface name="velocity"/>
+            </joint>
+            <joint name="omron/joint_5">
+                <command_interface name="position"/>
+                <state_interface name="position">
+                  <param name="initial_value">${initial_positions['omron/joint_5']}</param>
+                </state_interface>
+                <state_interface name="velocity"/>
+            </joint>
+            <joint name="omron/joint_6">
+                <command_interface name="position"/>
+                <state_interface name="position">
+                  <param name="initial_value">${initial_positions['omron/joint_6']}</param>
+                </state_interface>
+                <state_interface name="velocity"/>
+            </joint>
         </ros2_control>
     </xacro:macro>

Commit message: funzionagit add -Agit add -Agit add -Agit add -A! almeno la demo

File: battery_cell_description/urdf/battery_cell_rviz.xacro (robot description, xacro)
@@ -1,5 +1,5 @@
 <?xml version="1.0"?>
 <robot name="battery_cell" xmlns:xacro="http://www.ros.org/wiki/xacro">
-  <xacro:arg name="use_fake_hardware" default="false"/>
+  <xacro:arg name="use_fake_hardware" default="true"/>
   <xacro:property name="use_fake_hardware" value="'$(arg use_fake_hardware)'" />
   <link name="world"/>
@@ -24,6 +24,5 @@
   </joint>
   <xacro:include filename="$(find battery_cell_description)/urdf/comau_setup.xacro" />
-  <xacro:comau_setup use_fake_hardware="true"/>
-  <!-- <xacro:comau_setup use_fake_hardware="${use_fake_hardware}"/> -->
+  <xacro:comau_setup use_fake_hardware="${use_fake_hardware}"/>
   <joint name="world_to_comau" type="fixed">
       <origin

File: battery_cell_moveit_config/config/battery_cell.ros2_control.xacro (robot description, xacro)
@@ -2,5 +2,5 @@
 <robot xmlns:xacro="http://www.ros.org/wiki/xacro">
     <xacro:macro name="battery_cell_ros2_control" params="name initial_positions_file">
-        <xacro:property name="initial_positions" value="${load_yaml(initial_positions_file)['initial_positions']}"/>
+        <xacro:property name="initial_positions" value="${xacro.load_yaml(initial_positions_file)['initial_positions']}"/>
         <ros2_control name="${name}" type="system">
             <hardware>

Commit message: 2500Hz kuka ros2 controller config

File: battery_cell_description/urdf/battery_cell_rviz.xacro (robot description, xacro)
@@ -32,11 +32,11 @@
       <child link="comau_basement"/>
   </joint>
-  <xacro:include filename="$(find battery_cell_description)/urdf/omron_setup.xacro" />
-    <xacro:omron_setup use_fake_hardware="true"/>
+  <!-- <xacro:include filename="$(find battery_cell_description)/urdf/omron_setup.xacro" />
+    <xacro:omron_setup use_fake_hardware="true"/> -->
   <!-- <xacro:omron_setup use_fake_hardware="${use_fake_hardware}"/> -->
-  <joint name="world_to_map" type="fixed">
+  <!-- <joint name="world_to_map" type="fixed">
     <parent link="world"/>
     <child link="omron/map"/>
     <origin xyz="0.0 -4.0 0.0"/>
-  </joint>
+  </joint> -->
 </robot>

Commit message: working scaling

File: battery_cell_description/urdf/battery_cell_rviz.xacro (robot description, xacro)
@@ -32,11 +32,11 @@
       <child link="comau_basement"/>
   </joint>
-  <!-- <xacro:include filename="$(find battery_cell_description)/urdf/omron_setup.xacro" />
-    <xacro:omron_setup use_fake_hardware="true"/> -->
-  <!-- <xacro:omron_setup use_fake_hardware="${use_fake_hardware}"/> -->
-  <!-- <joint name="world_to_map" type="fixed">
+  <xacro:include filename="$(find battery_cell_description)/urdf/omron_setup.xacro" />
+  <!-- the real robot hardware_interface will be published by other means -->
+  <xacro:omron_setup use_fake_hardware="true"/>
+  <joint name="world_to_map" type="fixed">
     <parent link="world"/>
     <child link="omron/map"/>
     <origin xyz="0.0 -4.0 0.0"/>
-  </joint> -->
+  </joint>
 </robot>

Commit message: add launch arg include_omron

File: battery_cell_description/urdf/battery_cell_rviz.xacro (robot description, xacro)
@@ -2,4 +2,5 @@
 <robot name="battery_cell" xmlns:xacro="http://www.ros.org/wiki/xacro">
   <xacro:arg name="use_fake_hardware" default="true"/>
+  <xacro:arg name="include_omron" default="true"/>
   <xacro:property name="use_fake_hardware" value="'$(arg use_fake_hardware)'" />
   <link name="world"/>
@@ -32,11 +33,13 @@
       <child link="comau_basement"/>
   </joint>
-  <xacro:include filename="$(find battery_cell_description)/urdf/omron_setup.xacro" />
-  <!-- the real robot hardware_interface will be published by other means -->
-  <xacro:omron_setup use_fake_hardware="true"/>
-  <joint name="world_to_map" type="fixed">
-    <parent link="world"/>
-    <child link="omron/map"/>
-    <origin xyz="0.0 -4.0 0.0"/>
-  </joint>
+  <xacro:if value="$(arg include_omron)">
+    <xacro:include filename="$(find battery_cell_description)/urdf/omron_setup.xacro" />
+    <!-- the real robot hardware_interface will be published by other means -->
+    <xacro:omron_setup use_fake_hardware="true"/>
+    <joint name="world_to_map" type="fixed">
+      <parent link="world"/>
+      <child link="omron/map"/>
+      <origin xyz="0.0 -4.0 0.0"/>
+    </joint>
+  </xacro:if>
 </robot>

Commit message: wip

File: battery_cell_description/urdf/battery_cell_rviz.xacro (robot description, xacro)
@@ -40,5 +40,5 @@
       <parent link="world"/>
       <child link="omron/map"/>
-      <origin xyz="0.0 -4.0 0.0"/>
+      <origin xyz="3.80 0.52 0.0" rpy="0.0 0.0 -1.5707963267948966"/>
     </joint>
   </xacro:if>

Commit message: urdf updated

File: battery_cell_description/urdf/battery_cell_rviz.xacro (robot description, xacro)
@@ -23,8 +23,8 @@
       <child link="structure_base_link"/>
   </joint>
-  <xacro:include filename="$(find battery_cell_description)/urdf/battery_table.xacro" />
+  <!-- <xacro:include filename="$(find battery_cell_description)/urdf/battery_table.xacro" />
   <xacro:property name="table_prefix" value="'table_'" />
-  <xacro:battery_table prefix="${table_prefix}"/>
-  <joint name="world_to_table" type="fixed">
+  <xacro:battery_table prefix="${table_prefix}"/> -->
+  <!-- <joint name="world_to_table" type="fixed">
     <origin
       xyz="0.025 -1.58 0"
@@ -32,5 +32,95 @@
     <parent link="world"/>
     <child link="${table_prefix}base_link"/>
-  </joint>
+  </joint> -->
+  <!-- ## BATTERY HOLDER ## -->
+  <link name="battery_holder">
+    <visual>
+      <origin
+        xyz="0.0 0.0 0.0"/>
+      <geometry>
+        <mesh filename="package://battery_cell_description/meshes/battery_holder.STL"/>
+      </geometry>
+      <material
+        name="">
+        <color
+          rgba="0.5 0.5 0.5 1" />
+      </material>
+    </visual>
+    <collision>
+      <origin
+        xyz="0 0 0"
+        rpy="0 0 0" />
+      <geometry>
+        <mesh filename="package://battery_cell_description/meshes/battery_holder.STL"/>
+      </geometry>
+    </collision>
+  </link>
+  <joint name="world_to_bh" type="fixed">
+    <parent link="world"/>
+    <child link="battery_holder"/>
+    <origin xyz="1.3 -1.4 0"
+    rpy="1.57079632679489661923132169163975144209858469968 0 ${3.1415926535897932384626433832795028841971693993751058209749445923+0.5235987755982988}"/>
+  </joint>
+  <!-- ## - ## -->
+  <!-- ## Tools Kuka ## -->
+  <link name="kuka_tool_support">
+    <visual>
+      <origin
+        xyz="0.0 0.0 0.0"/>
+      <geometry>
+        <mesh filename="package://battery_cell_description/meshes/cambio_tool_kuka.STL"/>
+      </geometry>
+      <material
+        name="">
+        <color
+          rgba="0.5 0.5 0.5 1" />
+      </material>
+    </visual>
+    <collision>
+      <origin
+        xyz="0 0 0"
+        rpy="0 0 0" />
+      <geometry>
+        <mesh filename="package://battery_cell_description/meshes/cambio_tool_kuka.STL"/>
+      </geometry>
+    </collision>
+  </link>
+  <joint name="world_to_kuka_tools_support" type="fixed">
+    <parent link="world"/>
+    <child link="kuka_tool_support"/>
+    <origin xyz="0.8 0 0"
+    rpy="1.57079632679489661923132169163975144209858469968 0 0"/>
+  </joint>
+  <!-- ## - ## -->
+  <!-- ## Tools Comau ## -->
+  <link name="comau_tool_support">
+    <visual>
+      <origin
+        xyz="0.0 0.0 0.0"/>
+      <geometry>
+        <mesh filename="package://battery_cell_description/meshes/cambio_tool_comau.STL"/>
+      </geometry>
+      <material
+        name="">
+        <color
+          rgba="0.5 0.5 0.5 1" />
+      </material>
+    </visual>
+    <collision>
+      <origin
+        xyz="0 0 0"
+        rpy="0 0 0" />
+      <geometry>
+        <mesh filename="package://battery_cell_description/meshes/cambio_tool_comau.STL"/>
+      </geometry>
+    </collision>
+  </link>
+  <joint name="world_to_comau_tools_support" type="fixed">
+    <parent link="world"/>
+    <child link="comau_tool_support"/>
+    <origin xyz="-3.6 1.0 0.0"
+    rpy="1.57079632679489661923132169163975144209858469968 0 0"/>
+  </joint>
+  <!-- ## - ## -->
   <xacro:include filename="$(find battery_cell_description)/urdf/comau_setup.xacro" />
   <!-- <xacro:comau_setup use_fake_hardware="${use_fake_hardware}"/> -->
@@ -50,9 +140,8 @@
       <parent link="world"/>
       <child link="omron/map"/>
-      <origin xyz="3.80 0.52 0.0" rpy="0.0 0.0 -1.5707963267948966"/>
+      <!-- <origin xyz="3.80 0.52 0.0" rpy="0.0 0.0 -1.5707963267948966"/> -->
+      <origin xyz="-4.0 -1.640 0" rpy="0 0 0"/>
     </joint>
   </xacro:if>
-  <!-- <xacro:include filename="$(find battery_cell_description)/urdf/battery_cell_GPIO_ros2_control.xacro" />
-  <xacro:battery_cell_GPIO_ros2_control use_fake_hardware="$(arg use_GPIO_fake_hardware)"/> -->
   <!-- increased collisions -->
   <!-- FLOOR -->
@@ -250,8 +339,8 @@
   </joint>
   <!-- KUKA CONTROLLER BOX -->
-  <xacro:property name="kuka_controller_height" value="1.40" /> <!-- TODO -->
-  <xacro:property name="kuka_controller_length" value="1.20" /> <!-- TODO -->
-  <xacro:property name="kuka_controller_width" value="1.20" />  <!-- TODO -->
-  <link name="kuka_controller_link">
+  <!-- <xacro:property name="kuka_controller_height" value="1.40" /> TODO -->
+  <!-- <xacro:property name="kuka_controller_length" value="1.20" /> TODO -->
+  <!-- <xacro:property name="kuka_controller_width" value="1.20" />  TODO -->
+  <!-- <link name="kuka_controller_link">
     <inertial>
       <origin
@@ -293,8 +382,8 @@
     <origin
       xyz="-3.0 1.0 0.0"
-      rpy="0.0 0.0 0.0" />    <!-- TODO -->
+      rpy="0.0 0.0 0.0" />
     <parent link="structure_base_link"/>
     <child link="kuka_controller_link"/>
-  </joint>
+  </joint> -->
   <!-- end increased collisions -->
 </robot>

Commit message: add table

File: battery_cell_description/urdf/battery_cell_rviz.xacro (robot description, xacro)
@@ -23,14 +23,14 @@
       <child link="structure_base_link"/>
   </joint>
-  <!-- <xacro:include filename="$(find battery_cell_description)/urdf/battery_table.xacro" />
+  <xacro:include filename="$(find battery_cell_description)/urdf/battery_table.xacro" />
   <xacro:property name="table_prefix" value="'table_'" />
-  <xacro:battery_table prefix="${table_prefix}"/> -->
-  <!-- <joint name="world_to_table" type="fixed">
-    <origin
-      xyz="0.025 -1.58 0"
+  <xacro:battery_table prefix="${table_prefix}"/>
+  <joint name="world_to_table" type="fixed">
+    <origin
+      xyz="3.200 -0.25 0"
       rpy="0 0 0" />
     <parent link="world"/>
     <child link="${table_prefix}base_link"/>
-  </joint> -->
+  </joint>
   <!-- ## BATTERY HOLDER ## -->
   <link name="battery_holder">
