Commit message: z outgoing in base kuka

File: battery_cell_description/urdf/kuka_setup.xacro (robot description, xacro)
@@ -18,9 +18,25 @@
                        name="${prefix}${kuka_name}"
                        use_fake_hardware="${use_kuka_fake_hardware}" />
-    <joint name="kuka_structure_to_kr_50_r2500" type="fixed">
+    <link name="${prefix}${kuka_prefix}base_link_outgoing_z"/>
+    <joint name="kuka_structure_to_kr_outgoing_z" type="fixed">
         <origin
           xyz="0.333 -0.035 0.325"
+          rpy="${pi/2} 0 0" />
+        <parent link="${prefix}${kuka_structure_prefix}link_1"/>
+        <child link="${prefix}${kuka_prefix}base_link_outgoing_z"/>
+    </joint>
+    <link name="${prefix}${kuka_prefix}outgoing_z_to_base_link_tmp"/>
+    <joint name="outgoing_z_to_base_link_tmp_joint" type="fixed">
+        <origin
+          xyz="0 0 0"
           rpy="0 ${pi/2} 0" />
-        <parent link="${prefix}${kuka_structure_prefix}link_1"/>
+        <parent link="${prefix}${kuka_prefix}base_link_outgoing_z"/>
+        <child link="${prefix}${kuka_prefix}outgoing_z_to_base_link_tmp"/>
+    </joint>
+    <joint name="base_link_tmp_to_base_link_joint" type="fixed">
+        <origin
+          xyz="0 0 0"
+          rpy="0 0 -${pi/2}" />
+        <parent link="${prefix}${kuka_prefix}outgoing_z_to_base_link_tmp"/>
         <child link="${prefix}${kuka_prefix}base_link"/>
     </joint>

Commit message: update battery cell using the correct base_link of kuka

File: battery_cell_description/urdf/kuka_setup.xacro (robot description, xacro)
@@ -18,13 +18,12 @@
                        name="${prefix}${kuka_name}"
                        use_fake_hardware="${use_kuka_fake_hardware}" />
-    <link name="${prefix}${kuka_prefix}base_link_outgoing_z"/>
+    <!-- <link name="${prefix}${kuka_prefix}base_link_outgoing_z"/> -->
     <joint name="kuka_structure_to_kr_outgoing_z" type="fixed">
-        <origin
-          xyz="0.333 -0.035 0.325"
-          rpy="${pi/2} 0 0" />
-        <parent link="${prefix}${kuka_structure_prefix}link_1"/>
-        <child link="${prefix}${kuka_prefix}base_link_outgoing_z"/>
-    </joint>
-    <link name="${prefix}${kuka_prefix}outgoing_z_to_base_link_tmp"/>
+      <!-- <origin           xyz="0.333 -0.035 0.325"           rpy="${pi/2} 0 0" /> -->
+      <origin           xyz="0.333 -0.035 0.325"           rpy="0 0 0" />
+      <parent link="${prefix}${kuka_structure_prefix}link_1"/>
+        <child link="${prefix}${kuka_prefix}base_link"/>
+    </joint>
+    <!-- <link name="${prefix}${kuka_prefix}outgoing_z_to_base_link_tmp"/>
     <joint name="outgoing_z_to_base_link_tmp_joint" type="fixed">
         <origin
@@ -40,5 +39,5 @@
         <parent link="${prefix}${kuka_prefix}outgoing_z_to_base_link_tmp"/>
         <child link="${prefix}${kuka_prefix}base_link"/>
-    </joint>
+    </joint> -->
     <joint name="${prefix}${kuka_prefix}robot_to_sensor_flange1" type="fixed">
         <origin

Commit message: update urdf

File: battery_cell_description/urdf/kuka_setup.xacro (robot description, xacro)
@@ -21,5 +21,5 @@
     <joint name="kuka_structure_to_kr_outgoing_z" type="fixed">
       <!-- <origin           xyz="0.333 -0.035 0.325"           rpy="${pi/2} 0 0" /> -->
-      <origin           xyz="0.333 -0.035 0.325"           rpy="0 0 0" />
+      <origin           xyz="0.333 -0.035 0.325"           rpy="${pi/2} 0 0" />
       <parent link="${prefix}${kuka_structure_prefix}link_1"/>
         <child link="${prefix}${kuka_prefix}base_link"/>

Commit message: fix kuka rotation

File: battery_cell_description/urdf/kuka_setup.xacro (robot description, xacro)
@@ -21,5 +21,5 @@
     <joint name="kuka_structure_to_kr_outgoing_z" type="fixed">
       <!-- <origin           xyz="0.333 -0.035 0.325"           rpy="${pi/2} 0 0" /> -->
-      <origin           xyz="0.333 -0.035 0.325"           rpy="${pi/2} 0 0" />
+      <origin           xyz="0.333 -0.035 0.325"           rpy="${pi/2} ${pi/2} 0" />
       <parent link="${prefix}${kuka_structure_prefix}link_1"/>
         <child link="${prefix}${kuka_prefix}base_link"/>
