Commit message: End first gauss

File: battery_cell_description/urdf/battery_table.xacro (robot description, xacro)
@@ -11,5 +11,20 @@
   <xacro:property name="m_table" value="${steel_density*table_thickness*table_width*table_length}" />
   <xacro:property name="m_leg" value="${(m_tot - m_table) / 4}" />
-  <link name="${prefix}base_link"/>
+  <link name="${prefix}base_link">
+    <inertial>
+      <origin
+        xyz="0 0 0"
+        rpy="0 0 0" />
+      <mass
+        value="0.0001" />
+      <inertia
+        ixx="0.00000001"
+        ixy="0"
+        ixz="0"
+        iyy="0.00000001"
+        iyz="0"
+        izz="0.00000001" />
+    </inertial>
+  </link>
   <link name="${prefix}leg1_link">
     <inertial>

Commit message: Utils node added

File: battery_cell_description/urdf/battery_table.xacro (robot description, xacro)
@@ -2,5 +2,5 @@
 <robot name="battery_table" xmlns:xacro="http://www.ros.org/wiki/xacro">
 <xacro:macro name="battery_table" params="prefix:=''">
-  <xacro:property name="leg_height" value="0.900" />
+  <xacro:property name="leg_height" value="0.865" />
   <xacro:property name="leg_width" value="0.060" />
   <xacro:property name="table_thickness" value="0.015" />
@@ -11,5 +11,41 @@
   <xacro:property name="m_table" value="${steel_density*table_thickness*table_width*table_length}" />
   <xacro:property name="m_leg" value="${(m_tot - m_table) / 4}" />
-  <link name="${prefix}base_link"/>
+  <link name="${prefix}base_link">
+    <inertial>
+      <origin
+        xyz="0 0 0"
+        rpy="0 0 0" />
+      <mass
+        value="0.0001" />
+      <inertia
+        ixx="0.000001"
+        ixy="0"
+        ixz="0"
+        iyy="0.000001"
+        iyz="0"
+        izz="0.000001" />
+    </inertial>
+    <visual>
+      <origin
+        xyz="0 0 ${(leg_height+table_thickness)/2}"
+        rpy="0 0 0" />
+      <geometry>
+        <box size="${table_width+0.1} ${table_length+0.1} ${leg_height+table_thickness+0.1}"/>
+      </geometry>
+      <material
+        name="">
+        <color
+          rgba="0.1176 0.5059 0.6902 0.5" />
+      </material>
+    </visual>
+    <collision>
+      <origin
+        xyz="0 0 ${(leg_height+table_thickness)/2}"
+        rpy="0 0 0" />
+      <geometry>
+        <box size="${table_width} ${table_length} ${leg_height+table_thickness}"/>
+      </geometry>
+    </collision>
+  </link>
   <link name="${prefix}leg1_link">
     <inertial>
@@ -231,4 +267,51 @@
     <parent link="${prefix}base_link"/>
     <child link="${prefix}tabletop_link"/>
+  </joint>
+  <xacro:property name="battery_thickness" value="0.4" />
+  <xacro:property name="battery_width" value="${table_width}" />
+  <xacro:property name="battery_length" value="${table_length}" />
+  <link name="${prefix}battery_link">
+    <inertial>
+      <origin
+        xyz="0 0 0"
+        rpy="0 0 0" />
+      <mass
+        value="0.0001" />
+      <inertia
+        ixx="0.000001"
+        ixy="0"
+        ixz="0"
+        iyy="0.000001"
+        iyz="0"
+        izz="0.000001" />
+    </inertial>
+    <visual>
+      <origin
+        xyz="0 0 ${battery_thickness/2}"
+        rpy="0 0 0" />
+      <geometry>
+        <box size="${battery_width} ${battery_length} ${battery_thickness}"/>
+      </geometry>
+      <material
+        name="">
+        <color
+          rgba="0.1176 0.5059 0.6902 0.5" />
+      </material>
+    </visual>
+    <collision>
+      <origin
+        xyz="0 0 ${battery_thickness/2}"
+        rpy="0 0 0" />
+      <geometry>
+        <box size="${battery_width} ${battery_length} ${battery_thickness}"/>
+      </geometry>
+    </collision>
+  </link>
+  <joint name="${prefix}base_to_battery" type="fixed">
+    <origin
+      xyz="0 0 ${leg_height+table_thickness}"
+      rpy="0 0 0" />
+    <parent link="${prefix}base_link"/>
+    <child link="${prefix}battery_link"/>
   </joint>
 </xacro:macro>

Commit message: ready for tests

File: battery_cell_description/urdf/battery_table.xacro (robot description, xacro)
@@ -1,235 +1,466 @@
 <?xml version="1.0"?>
 <robot name="battery_table" xmlns:xacro="http://www.ros.org/wiki/xacro">
-<xacro:macro name="battery_table" params="prefix:=''">
-  <xacro:property name="leg_height" value="0.900" />
-  <xacro:property name="leg_width" value="0.060" />
-  <xacro:property name="table_thickness" value="0.015" />
-  <xacro:property name="table_width" value="1.500" />
-  <xacro:property name="table_length" value="1.480" />
-  <xacro:property name="steel_density" value="7859.0" /> <!-- tabletop material: S355J2+N steel (density in kg/m^3) -->
-  <xacro:property name="m_tot" value="300.0" />
-  <xacro:property name="m_table" value="${steel_density*table_thickness*table_width*table_length}" />
-  <xacro:property name="m_leg" value="${(m_tot - m_table) / 4}" />
-  <link name="${prefix}base_link"/>
-  <link name="${prefix}leg1_link">
-    <inertial>
-      <origin
-        xyz="0 0 ${leg_height/2}"
-        rpy="0 0 0" />
-      <mass
-        value="${m_leg}" />
-      <inertia
-        ixx="${1/12*m_leg*(leg_width*leg_width + leg_height*leg_height)}"
-        ixy="0"
-        ixz="0"
-        iyy="${1/12*m_leg*(leg_width*leg_width + leg_height*leg_height)}"
-        iyz="0"
-        izz="${1/12*m_leg*(leg_width*leg_width + leg_width*leg_width)}" />
-    </inertial>
-    <visual>
-      <origin
-        xyz="0 0 ${leg_height/2}"
-        rpy="0 0 0" />
-      <geometry>
-        <box size="${leg_width} ${leg_width} ${leg_height}"/>
-      </geometry>
-      <material
-        name="">
-        <color
-          rgba="0.1176 0.5059 0.6902 1" />
-      </material>
-    </visual>
-    <collision>
-      <origin
-        xyz="0 0 ${leg_height/2}"
-        rpy="0 0 0" />
-      <geometry>
-        <box size="${leg_width} ${leg_width} ${leg_height}"/>
-      </geometry>
-    </collision>
-  </link>
-  <joint name="${prefix}base_to_leg1" type="fixed">
-    <origin
-      xyz="${table_width/2-leg_width/2} ${table_length/2-leg_width/2} 0"
-      rpy="0 0 0" />
-    <parent link="${prefix}base_link"/>
-    <child link="${prefix}leg1_link"/>
-  </joint>
-  <link name="${prefix}leg2_link">
-    <inertial>
-      <origin
-        xyz="0 0 ${leg_height/2}"
-        rpy="0 0 0" />
-      <mass
-        value="${m_leg}" />
-      <inertia
-        ixx="${1/12*m_leg*(leg_width*leg_width + leg_height*leg_height)}"
-        ixy="0"
-        ixz="0"
-        iyy="${1/12*m_leg*(leg_width*leg_width + leg_height*leg_height)}"
-        iyz="0"
-        izz="${1/12*m_leg*(leg_width*leg_width + leg_width*leg_width)}" />
-    </inertial>
-    <visual>
-      <origin
-        xyz="0 0 ${leg_height/2}"
-        rpy="0 0 0" />
-      <geometry>
-        <box size="${leg_width} ${leg_width} ${leg_height}"/>
-      </geometry>
-      <material
-        name="">
-        <color
-          rgba="0.1176 0.5059 0.6902 1" />
-      </material>
-    </visual>
-    <collision>
-      <origin
-        xyz="0 0 ${leg_height/2}"
-        rpy="0 0 0" />
-      <geometry>
-        <box size="${leg_width} ${leg_width} ${leg_height}"/>
-      </geometry>
-    </collision>
-  </link>
-  <joint name="${prefix}base_to_leg2" type="fixed">
-    <origin
-      xyz="${table_width/2-leg_width/2} ${-table_length/2+leg_width/2} 0"
-      rpy="0 0 0" />
-    <parent link="${prefix}base_link"/>
-    <child link="${prefix}leg2_link"/>
-  </joint>
-  <link name="${prefix}leg3_link">
-    <inertial>
-      <origin
-        xyz="0 0 ${leg_height/2}"
-        rpy="0 0 0" />
-      <mass
-        value="${m_leg}" />
-      <inertia
-        ixx="${1/12*m_leg*(leg_width*leg_width + leg_height*leg_height)}"
-        ixy="0"
-        ixz="0"
-        iyy="${1/12*m_leg*(leg_width*leg_width + leg_height*leg_height)}"
-        iyz="0"
-        izz="${1/12*m_leg*(leg_width*leg_width + leg_width*leg_width)}" />
-    </inertial>
-    <visual>
-      <origin
-        xyz="0 0 ${leg_height/2}"
-        rpy="0 0 0" />
-      <geometry>
-        <box size="${leg_width} ${leg_width} ${leg_height}"/>
-      </geometry>
-      <material
-        name="">
-        <color
-          rgba="0.1176 0.5059 0.6902 1" />
-      </material>
-    </visual>
-    <collision>
-      <origin
-        xyz="0 0 ${leg_height/2}"
-        rpy="0 0 0" />
-      <geometry>
-        <box size="${leg_width} ${leg_width} ${leg_height}"/>
-      </geometry>
-    </collision>
-  </link>
-  <joint name="${prefix}base_to_leg3" type="fixed">
-    <origin
-      xyz="${-table_width/2+leg_width/2} ${-table_length/2+leg_width/2} 0"
-      rpy="0 0 0" />
-    <parent link="${prefix}base_link"/>
-    <child link="${prefix}leg3_link"/>
-  </joint>
-  <link name="${prefix}leg4_link">
-    <inertial>
-      <origin
-        xyz="0 0 ${leg_height/2}"
-        rpy="0 0 0" />
-      <mass
-        value="${m_leg}" />
-      <inertia
-        ixx="${1/12*m_leg*(leg_width*leg_width + leg_height*leg_height)}"
-        ixy="0"
-        ixz="0"
-        iyy="${1/12*m_leg*(leg_width*leg_width + leg_height*leg_height)}"
-        iyz="0"
-        izz="${1/12*m_leg*(leg_width*leg_width + leg_width*leg_width)}" />
-    </inertial>
-    <visual>
-      <origin
-        xyz="0 0 ${leg_height/2}"
-        rpy="0 0 0" />
-      <geometry>
-        <box size="${leg_width} ${leg_width} ${leg_height}"/>
-      </geometry>
-      <material
-        name="">
-        <color
-          rgba="0.1176 0.5059 0.6902 1" />
-      </material>
-    </visual>
-    <collision>
-      <origin
-        xyz="0 0 ${leg_height/2}"
-        rpy="0 0 0" />
-      <geometry>
-        <box size="${leg_width} ${leg_width} ${leg_height}"/>
-      </geometry>
-    </collision>
-  </link>
-  <joint name="${prefix}base_to_leg4" type="fixed">
-    <origin
-      xyz="${-table_width/2+leg_width/2} ${table_length/2-leg_width/2} 0"
-      rpy="0 0 0" />
-    <parent link="${prefix}base_link"/>
-    <child link="${prefix}leg4_link"/>
-  </joint>
-  <link name="${prefix}tabletop_link">
-    <inertial>
-      <origin
-        xyz="0 0 ${table_thickness/2}"
-        rpy="0 0 0" />
-      <mass
-        value="${m_leg}" />
-      <inertia
-        ixx="${1/12*m_table*(table_length*table_length + table_thickness*table_thickness)}"
-        ixy="0"
-        ixz="0"
-        iyy="${1/12*m_table*(table_width*table_width + table_thickness*table_thickness)}"
-        iyz="0"
-        izz="${1/12*m_table*(table_width*table_width + table_length*table_length)}" />
-    </inertial>
-    <visual>
-      <origin
-        xyz="0 0 ${table_thickness/2}"
-        rpy="0 0 0" />
-      <geometry>
-        <box size="${table_width} ${table_length} ${table_thickness}"/>
-      </geometry>
-      <material
-        name="">
-        <color
-          rgba="0.6608 0.6608 0.7878 1" />
-      </material>
-    </visual>
-    <collision>
-      <origin
-        xyz="0 0 ${table_thickness/2}"
-        rpy="0 0 0" />
-      <geometry>
-        <box size="${table_width} ${table_length} ${table_thickness}"/>
-      </geometry>
-    </collision>
-  </link>
-  <joint name="${prefix}base_to_tabletop" type="fixed">
-    <origin
-      xyz="0 0 ${leg_height}"
-      rpy="0 0 0" />
-    <parent link="${prefix}base_link"/>
-    <child link="${prefix}tabletop_link"/>
-  </joint>
-</xacro:macro>
+  <xacro:macro name="battery_table" params="prefix:='' type:='rviz'">
+    <xacro:property name="leg_height" value="0.94" />
+    <xacro:property name="leg_width" value="0.060" />
+    <xacro:property name="table_thickness" value="0.015" />
+    <xacro:property name="table_width" value="1.500" />
+    <xacro:property name="table_length" value="1.480" />
+    <xacro:property name="steel_density" value="7859.0" /> <!-- tabletop material: S355J2+N steel (density in kg/m^3) -->
+    <xacro:property name="m_tot" value="300.0" />
+    <xacro:property name="m_table" value="${steel_density*table_thickness*table_width*table_length}" />
+    <xacro:property name="m_leg" value="${(m_tot - m_table) / 4}" />
+    <xacro:if value="${type == 'rviz'}">
+      <link name="${prefix}base_link">
+        <inertial>
+          <origin
+            xyz="0 0 0"
+            rpy="0 0 0" />
+          <mass
+            value="0.0001" />
+          <inertia
+            ixx="0.000001"
+            ixy="0"
+            ixz="0"
+            iyy="0.000001"
+            iyz="0"
+            izz="0.000001" />
+        </inertial>
+        <!-- <visual>
+          <origin
+            xyz="0 0 ${(leg_height+table_thickness)/2}"
+            rpy="0 0 0" />
+          <geometry>
+            <box size="${table_width+0.1} ${table_length+0.1} ${leg_height+table_thickness+0.1}"/>
+          </geometry>
+          <material
+            name="">
+            <color
+              rgba="0.1176 0.5059 0.6902 0.5" />
+          </material>
+        </visual>
+        <collision>
+          <origin
+            xyz="0 0 ${(leg_height+table_thickness)/2}"
+            rpy="0 0 0" />
+          <geometry>
+            <box size="${table_width} ${table_length} ${leg_height+table_thickness}"/>
+          </geometry>
+        </collision> -->
+      </link>
+    </xacro:if>
+    <xacro:unless value="${type == 'rviz'}">
+      <link name="${prefix}base_link">
+        <inertial>
+          <origin
+            xyz="0 0 0"
+            rpy="0 0 0" />
+          <mass
+            value="0.0001" />
+          <inertia
+            ixx="0.000001"
+            ixy="0"
+            ixz="0"
+            iyy="0.000001"
+            iyz="0"
+            izz="0.000001" />
+        </inertial>
+      </link>
+    </xacro:unless>
+    <link name="${prefix}leg1_link">
+      <inertial>
+        <origin
+          xyz="0 0 ${leg_height/2}"
+          rpy="0 0 0" />
+        <mass
+          value="${m_leg}" />
+        <inertia
+          ixx="${1/12*m_leg*(leg_width*leg_width + leg_height*leg_height)}"
+          ixy="0"
+          ixz="0"
+          iyy="${1/12*m_leg*(leg_width*leg_width + leg_height*leg_height)}"
+          iyz="0"
+          izz="${1/12*m_leg*(leg_width*leg_width + leg_width*leg_width)}" />
+      </inertial>
+      <visual>
+        <origin
+          xyz="0 0 ${leg_height/2}"
+          rpy="0 0 0" />
+        <geometry>
+          <box size="${leg_width} ${leg_width} ${leg_height}"/>
+        </geometry>
+        <material
+          name="">
+          <color
+            rgba="0.1176 0.5059 0.6902 1" />
+        </material>
+      </visual>
+      <collision>
+        <origin
+          xyz="0 0 ${leg_height/2}"
+          rpy="0 0 0" />
+        <geometry>
+          <box size="${leg_width} ${leg_width} ${leg_height}"/>
+        </geometry>
+      </collision>
+    </link>
+    <joint name="${prefix}base_to_leg1" type="fixed">
+      <origin
+        xyz="${table_width/2-leg_width/2} ${table_length/2-leg_width/2} 0"
+        rpy="0 0 0" />
+      <parent link="${prefix}base_link"/>
+      <child link="${prefix}leg1_link"/>
+    </joint>
+    <link name="${prefix}leg2_link">
+      <inertial>
+        <origin
+          xyz="0 0 ${leg_height/2}"
+          rpy="0 0 0" />
+        <mass
+          value="${m_leg}" />
+        <inertia
+          ixx="${1/12*m_leg*(leg_width*leg_width + leg_height*leg_height)}"
+          ixy="0"
+          ixz="0"
+          iyy="${1/12*m_leg*(leg_width*leg_width + leg_height*leg_height)}"
+          iyz="0"
+          izz="${1/12*m_leg*(leg_width*leg_width + leg_width*leg_width)}" />
+      </inertial>
+      <visual>
+        <origin
+          xyz="0 0 ${leg_height/2}"
+          rpy="0 0 0" />
+        <geometry>
+          <box size="${leg_width} ${leg_width} ${leg_height}"/>
+        </geometry>
+        <material
+          name="">
+          <color
+            rgba="0.1176 0.5059 0.6902 1" />
+        </material>
+      </visual>
+      <collision>
+        <origin
+          xyz="0 0 ${leg_height/2}"
+          rpy="0 0 0" />
+        <geometry>
+          <box size="${leg_width} ${leg_width} ${leg_height}"/>
+        </geometry>
+      </collision>
+    </link>
+    <joint name="${prefix}base_to_leg2" type="fixed">
+      <origin
+        xyz="${table_width/2-leg_width/2} ${-table_length/2+leg_width/2} 0"
+        rpy="0 0 0" />
+      <parent link="${prefix}base_link"/>
+      <child link="${prefix}leg2_link"/>
+    </joint>
+    <link name="${prefix}leg3_link">
+      <inertial>
+        <origin
+          xyz="0 0 ${leg_height/2}"
+          rpy="0 0 0" />
+        <mass
+          value="${m_leg}" />
+        <inertia
+          ixx="${1/12*m_leg*(leg_width*leg_width + leg_height*leg_height)}"
+          ixy="0"
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