Commit message: ready for tests

File: battery_cell_moveit_config/config/gazebo_battery_cell.urdf (robot description, URDF)
Before this commit: robot battery_cell, 65 links, 64 joints
Links:
- removed link kr_base_link
- removed link kr_closed_tip
- removed link kr_flange
- removed link kr_gripper_base
- removed link kr_left_base_rod
- removed link kr_left_crank
- removed link kr_left_external_crank
- removed link kr_left_phalanx
- removed link kr_left_rod
- removed link kr_link1
- removed link kr_link2
- removed link kr_link3
- removed link kr_link4
- removed link kr_link5
- removed link kr_link6
- removed link kr_open_tip
- removed link kr_right_base_rod
- removed link kr_right_crank
- removed link kr_right_external_crank
- removed link kr_right_phalanx
- removed link kr_right_rod
- removed link kr_zero_pos_tip
- removed link nj_base_link
- removed link nj_external_piece
- removed link nj_flange
- removed link nj_link_1
- removed link nj_link_2
- removed link nj_link_2_1
- removed link nj_link_2_2
- removed link nj_link_2_2_virtual
- removed link nj_link_2_3
- removed link nj_link_2_4
- removed link nj_link_3
- removed link nj_link_3_virtual
- removed link nj_link_4
- removed link nj_link_5
- removed link nj_link_6
- removed link nj_motor_1
- removed link nj_motor_2
- removed link nj_motor_3
- removed link nj_motor_4
- removed link nj_motor_5
- removed link nj_motor_6
- removed link omron_agv_base_link
- removed link omron_arm_base_link
- removed link omron_arm_flange
- removed link omron_arm_link_0
- removed link omron_arm_link_1
- removed link omron_arm_link_2
- removed link omron_arm_link_3
- removed link omron_arm_link_4
- removed link omron_arm_link_5
- removed link omron_arm_link_6
- removed link omron_base_link
- removed link omron_base_x
- removed link omron_base_y
- added link comau_basement, mass 10000; collision box size=1.11 1.01 0.028; visual box size=1.11 1.01 0.028
- added link comau_fake_robot, mass 10000; collision box size=2 3 3; visual box size=2 3 3
- added link gripper_base, mass 0.6818; collision mesh filename=package://schunk_gripper_jpg_p_160_description/meshes/SCHUN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; visual mesh filename=package://schunk_gripper_jpg_p_160_description/meshes/SCHUN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
- added link gripper_end_left_circle, mass 0.0001; visual box size=0.01 0.05 0.01
- added link gripper_end_right_circle, mass 0.0001; visual box size=0.01 0.05 0.01
- added link gripper_left_circle, mass 0.0001
- added link gripper_left_finger, mass 0.10; collision mesh filename=package://schunk_gripper_jpg_p_160_description/meshes/Finge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; visual mesh filename=package://schunk_gripper_jpg_p_160_description/meshes/Finge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
- added link gripper_left_slider, mass 0.070; collision mesh filename=package://schunk_gripper_jpg_p_160_description/meshes/SCHUN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; visual mesh filename=package://schunk_gripper_jpg_p_160_description/meshes/SCHUN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
- added link gripper_middle_left_circle, mass 0.0001
- added link gripper_middle_right_circle, mass 0.0001
- added link gripper_right_circle, mass 0.0001
- added link gripper_right_finger, mass 0.10; collision mesh filename=package://schunk_gripper_jpg_p_160_description/meshes/Finge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; visual mesh filename=package://schunk_gripper_jpg_p_160_description/meshes/Finge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
- added link gripper_right_slider, mass 0.070; collision mesh filename=package://schunk_gripper_jpg_p_160_description/meshes/SCHUN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; visual mesh filename=package://schunk_gripper_jpg_p_160_description/meshes/SCHUN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
- added link gripper_working_point
- added link kuka_base_link, mass 30.385; collision mesh filename=package://kr_50_r2500_description/meshes/base_link.STL; visual mesh filename=package://kr_50_r2500_description/meshes/base_link.STL
- added link kuka_flange, mass 0.01
- added link kuka_gripper_flange, mass 0.12657298; collision mesh filename=package://schunk_gripper_jpg_p_160_description/meshes/senso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; visual mesh filename=package://schunk_gripper_jpg_p_160_description/meshes/senso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
- added link kuka_link1, mass 56.0953515273858; collision mesh filename=package://kr_50_r2500_description/meshes/link1.STL; visual mesh filename=package://kr_50_r2500_description/meshes/link1.STL
- added link kuka_link2, mass 35.5942562362571; collision mesh filename=package://kr_50_r2500_description/meshes/link2.STL; visual mesh filename=package://kr_50_r2500_description/meshes/link2.STL
- added link kuka_link3, mass 36.6784876951283; collision mesh filename=package://kr_50_r2500_description/meshes/link3.STL; visual mesh filename=package://kr_50_r2500_description/meshes/link3.STL
- added link kuka_link4, mass 15.1542881051753; collision mesh filename=package://kr_50_r2500_description/meshes/link4.STL; visual mesh filename=package://kr_50_r2500_description/meshes/link4.STL
- added link kuka_link5, mass 5.17490767884354; collision mesh filename=package://kr_50_r2500_description/meshes/link5.STL; visual mesh filename=package://kr_50_r2500_description/meshes/link5.STL
- added link kuka_link6, mass 0.362972835401582; collision mesh filename=package://kr_50_r2500_description/meshes/link6.STL; visual mesh filename=package://kr_50_r2500_description/meshes/link6.STL
- added link kuka_sensor, mass 0.169; collision mesh filename=package://battery_cell_description/meshes/sensor.STL; visual mesh filename=package://battery_cell_description/meshes/sensor.STL
- added link kuka_sensor_flange1, mass 0.365; collision mesh filename=package://battery_cell_description/meshes/sensor_flange_rob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; visual mesh filename=package://battery_cell_description/meshes/sensor_flange_rob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
- added link kuka_sensor_flange2, mass 0.337; collision mesh filename=package://battery_cell_description/meshes/sensor_flange_sen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; visual mesh filename=package://battery_cell_description/meshes/sensor_flange_sen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
- added link structure_fake_structure, mass 10000; collision box size=4.3 1.5 4.0; visual box size=4.3 1.5 4.0
- added link structure_fake_structure_left_foot, mass 10000; collision box size=0.87 1.5 1.3; visual box size=0.87 1.5 1.3
- added link structure_fake_structure_right_foot, mass 10000; collision box size=0.87 1.5 1.3; visual box size=0.87 1.5 1.3
- added link table_can_hole, mass 0.0001; collision mesh filename=package://battery_cell_description/meshes/Hole_60.STL; visual mesh filename=package://battery_cell_description/meshes/Hole_60.STL
- added link table_fake_plane, mass 0.0001; collision box size=10 10 0.02; visual box size=10 10 0.03
- added link table_fake_wall, mass 0.0001; collision box size=3 0.02 2; visual box size=3 0.02 2
- added link table_vertex0
- added link table_vertex1
- added link table_vertex2
- added link table_vertex3
- added link table_vertex4
- link structure_base_link: geometry collision mesh filename=package://kuka_structure_description/meshes/base_link.STL scale=0.001 0.001 0.001; visual mesh filename=package://kuka_structure_description/meshes/base_link.STL scale=0.001 0.001 0.001
- link structure_link_1: geometry collision mesh filename=package://kuka_structure_description/meshes/link_1.STL scale=0.001 0.001 0.001; visual mesh filename=package://kuka_structure_description/meshes/link_1.STL scale=0.001 0.001 0.001
- link table_base_link: mass None -> 0.0001
- link table_leg1_link: geometry collision box size=0.06 0.06 0.94; visual box size=0.06 0.06 0.94
- link table_leg2_link: geometry collision box size=0.06 0.06 0.94; visual box size=0.06 0.06 0.94
- link table_leg3_link: geometry collision box size=0.06 0.06 0.94; visual box size=0.06 0.06 0.94
- link table_leg4_link: geometry collision box size=0.06 0.06 0.94; visual box size=0.06 0.06 0.94
Joints:
- removed joint kr_closed_tip_joint
- removed joint kr_gripper_joint
- removed joint kr_joint1
- removed joint kr_joint2
- removed joint kr_joint3
- removed joint kr_joint4
- removed joint kr_joint5
- removed joint kr_joint6
- removed joint kr_left_finger_joint
- removed joint kr_left_joint_1_2
- removed joint kr_left_joint_2_3
- removed joint kr_left_joint_2_5
- removed joint kr_left_joint_3_4
- removed joint kr_link6_to_flange
- removed joint kr_open_tip_joint
- removed joint kr_right_finger_joint
- removed joint kr_right_joint_1_2
- removed joint kr_right_joint_2_3
- removed joint kr_right_joint_2_5
- removed joint kr_right_joint_3_4
- removed joint kr_zero_pos_tip_joint
- removed joint nj_joint_1
- removed joint nj_joint_2
- removed joint nj_joint_2_1
- removed joint nj_joint_2_2
- removed joint nj_joint_2_3
- removed joint nj_joint_2_4
- removed joint nj_joint_2m
- removed joint nj_joint_3
- removed joint nj_joint_3m
- removed joint nj_joint_4
- removed joint nj_joint_5
- removed joint nj_joint_6
- removed joint nj_joint_external_piece
- removed joint nj_joint_motor_1
- removed joint nj_joint_motor_2
- removed joint nj_joint_motor_3
- removed joint nj_joint_motor_4
- removed joint nj_joint_motor_5
- removed joint nj_joint_motor_6
- removed joint nj_link_6_to_flange
- removed joint omron_arm_base_fixed_joint
- removed joint omron_arm_flange_fixed_joint
- removed joint omron_arm_joint_1
- removed joint omron_arm_joint_2
- removed joint omron_arm_joint_3
- removed joint omron_arm_joint_4
- removed joint omron_arm_joint_5
- removed joint omron_arm_joint_6
- removed joint omron_joint_rev
- removed joint omron_joint_x
- removed joint omron_joint_y
- removed joint omron_lifter
- removed joint world_to_kuka_structure
- removed joint world_to_nj_220_2_7
- removed joint world_to_omron
- added joint comau_fake_robot: type fixed, parent comau_basement, child comau_fake_robot, origin xyz=-0.05 -0.05 0.028 rpy=0 0 0
- added joint gripper_end_left_joint_circle: type revolute, parent gripper_middle_left_circle, child gripper_end_left_circle, origin xyz=0.0 0.0 0.0 rpy=0 0 0, axis 0 1 0, limit lower=-200 upper=200 effort=1000 velocity=1000
- added joint gripper_end_right_joint_circle: type revolute, parent gripper_middle_right_circle, child gripper_end_right_circle, origin xyz=0.0 0.0 0.0 rpy=0 0 0, axis 0 1 0, limit lower=-200 upper=200 effort=1000 velocity=1000
- added joint gripper_joint: type fixed, parent kuka_gripper_flange, child gripper_base, origin xyz=0 0 0.015 rpy=0 0 0
- added joint gripper_left_finger_joint: type fixed, parent gripper_left_slider, child gripper_left_finger, origin xyz=0.0285 0 0.0289 rpy=0 0 3.14159, axis 0 0 0
- added joint gripper_left_joint: type prismatic, parent gripper_base, child gripper_left_slider, origin xyz=0.0006 0 0.0481 rpy=0 0 0, axis 1 0 0, limit lower=0.000 upper=0.017 effort=1000 velocity=1000000, mimic joint=gripper_left_joint_circle multiplier=0.05 offset=-0.00086
- added joint gripper_left_joint_circle: type revolute, parent gripper_base, child gripper_left_circle, origin xyz=0.0 0.0 0.0 rpy=0 0.0 0, axis 0 1 0, limit lower=-100 upper=100 effort=10000 velocity=1000
- added joint gripper_middle_left_joint_circle: type prismatic, parent gripper_left_circle, child gripper_middle_left_circle, origin xyz=0 0 0 rpy=0 0 0, axis 0 0 1, limit lower=-1 upper=1 effort=10000 velocity=1000
- added joint gripper_middle_right_joint_circle: type prismatic, parent gripper_right_circle, child gripper_middle_right_circle, origin xyz=0 0 0 rpy=0 0 0, axis 0 0 1, limit lower=-1 upper=1 effort=10000 velocity=1000
- added joint gripper_right_finger_joint: type fixed, parent gripper_right_slider, child gripper_right_finger, origin xyz=0.0285 0 0.0289 rpy=0 0 3.14159, axis 0 0 0
- added joint gripper_right_joint: type prismatic, parent gripper_base, child gripper_right_slider, origin xyz=-0.0006 0 0.0481 rpy=0 0 3.14159, axis 1 0 0, limit lower=0.000 upper=0.017 effort=100000 velocity=1000000, mimic joint=gripper_left_joint multiplier=1 offset=0
- added joint gripper_right_joint_circle: type revolute, parent gripper_base, child gripper_right_circle, origin xyz=0.0 0.0 0.0 rpy=0 0.0 0, axis 0 1 0, limit lower=-100 upper=100 effort=10000 velocity=1000
- added joint gripper_working_point_joint: type fixed, parent gripper_base, child gripper_working_point, origin xyz=0.0 0 0.163 rpy=0 0 0, axis 0 0 0
- added joint kuka_fake_structure: type fixed, parent structure_base_link, child structure_fake_structure, origin xyz=-0.45 0.2  0 rpy=0 0 0
- added joint kuka_fake_structure_left_foot: type fixed, parent structure_base_link, child structure_fake_structure_left_foot, origin xyz=2.45 -0.05  0 rpy=0 0 0
- added joint kuka_fake_structure_right_foot: type fixed, parent structure_base_link, child structure_fake_structure_right_foot, origin xyz=-0.05 -0.05 0 rpy=0 0 0
- added joint kuka_joint1: type revolute, parent kuka_base_link, child kuka_link1, origin xyz=0 -0.17 0 rpy=1.5708 0.009141 0, axis 0 0 -1, limit lower=-3.22886 upper=3.22886 effort=10000 velocity=3.05433
- added joint kuka_joint2: type revolute, parent kuka_link1, child kuka_link2, origin xyz=0.175 -0.074807 0.405 rpy=0 1.557055  0, axis 0 1 0, limit lower=-3.05433 upper=1.0472 effort=10000 velocity=2.75762
- added joint kuka_joint3: type revolute, parent kuka_link2, child kuka_link3, origin xyz=0 0 1.29 rpy=0 -1.557055 0, axis 0 1 0, limit lower=-2.0944 upper=2.96706 effort=10000 velocity=3.05433
- added joint kuka_joint4: type revolute, parent kuka_link3, child kuka_link4, origin xyz=0.32687 0.074807 0.05 rpy=0 0 0, axis -1 0 0, limit lower=-2.79253 upper=2.79253 effort=10000 velocity=4.36332
- added joint kuka_joint5: type revolute, parent kuka_link4, child kuka_link5, origin xyz=0.708131634616243 0 0 rpy=0 -0.0 0, axis 0 1 0, limit lower=-2.18166 upper=2.18166 effort=10000 velocity=4.36332
- added joint kuka_joint6: type revolute, parent kuka_link5, child kuka_link6, origin xyz=0.0966663727881543 0 0 rpy=0 0 0, axis -1 0 0, limit lower=-3.31613 upper=3.31613 effort=10000 velocity=6.28319
- added joint kuka_link6_to_flange: type fixed, parent kuka_link6, child kuka_flange, origin xyz=0.07 0 0 rpy=0 1.57079632679 0
- added joint kuka_robot_to_sensor_flange1: type fixed, parent kuka_flange, child kuka_sensor_flange1, origin xyz=0 0 0 rpy=0 0 1.5708
- added joint kuka_sensor_flange1_sensor_flange2: type fixed, parent kuka_sensor_flange1, child kuka_sensor_flange2, origin xyz=0 0 0.02 rpy=0 0 0
- added joint kuka_sensor_flange2_to_sensor: type fixed, parent kuka_sensor_flange2, child kuka_sensor, origin xyz=0 0 0.02 rpy=0 0 0
- added joint kuka_sensor_to_gripper_flange: type fixed, parent kuka_sensor, child kuka_gripper_flange, origin xyz=0 0 0.0286 rpy=0 0 0
- added joint table_base_to_plane: type fixed, parent table_base_link, child table_fake_plane, origin xyz=0 0 0.955 rpy=0 0 0
- added joint table_base_to_wall: type fixed, parent table_base_link, child table_fake_wall, origin xyz=0 -0.40 0.5 rpy=0 0 0
- added joint table_tabletop_to_hole: type fixed, parent table_tabletop_link, child table_can_hole, origin xyz=0.65 0.35 0.015 rpy=0 0 0
- added joint table_vertex0: type fixed, parent table_tabletop_link, child table_vertex0, origin xyz=0 0 0 rpy=0 0 0
- added joint table_vertex1: type fixed, parent table_tabletop_link, child table_vertex1, origin xyz=0.75 0.74 0 rpy=0 0 0
- added joint table_vertex2: type fixed, parent table_tabletop_link, child table_vertex2, origin xyz=0.75 -0.74 0 rpy=0 0 0
- added joint table_vertex3: type fixed, parent table_tabletop_link, child table_vertex3, origin xyz=-0.75 0.74 0 rpy=0 0 0
- added joint table_vertex4: type fixed, parent table_tabletop_link, child table_vertex4, origin xyz=-0.75 -0.74 0 rpy=0 0 0
- added joint world_to_comau: type fixed, parent world, child comau_basement, origin xyz=-2.708 -0.430 0 rpy=0 0 3.14159
- added joint world_to_kuka: type fixed, parent world, child structure_base_link, origin xyz=0 0 0 rpy=0 0 0
- joint kuka_structure_to_kr_50_r2500: child kr_base_link -> kuka_base_link
- joint structure_joint_1: axis -1 0 0 -> 1 0 0; limit lower=0 upper=3.0 effort=100000 velocity=1.74533 -> lower=0 upper=2.9 effort=100000 velocity=1.74533; origin xyz=2.750 0.215 2.720 rpy=0 0 0 -> xyz=-0.250 0.215 2.720 rpy=0 0 0; type prismatic -> fixed
- joint table_base_to_tabletop: origin xyz=0 0 0.9 rpy=0 0 0 -> xyz=0 0 0.94 rpy=0 0 0
- joint world_to_table: origin xyz=1 -1 0 rpy=0 0 0 -> xyz=0.051 -1.61 0 rpy=0 0 -0.015

Commit message: Removed last mergh problem

File: battery_cell_description/urdf/battery_table.xacro (robot description, xacro)
@@ -463,9 +463,4 @@
       </joint>
    </xacro:if>
-<<<<<<< HEAD
   </xacro:macro>
 </robot>
-=======
-</xacro:macro>
-</robot>
->>>>>>> 4cf6f8cb3c5076118f2ddc0fe4f8ab67712ee64f

Commit message: birmingham adaptation

File: battery_cell_description/urdf/battery_table.xacro (robot description, xacro)
@@ -353,5 +353,4 @@
             rpy="0 0 0" />
           <geometry>
-            <!-- <box size="10 10 0.02"/> -->
             <box size="10 10 0.03"/>
           </geometry>
@@ -422,5 +421,5 @@
         <child link="${prefix}fake_wall"/>
       </joint>
-      <link name="${prefix}vertex0"/>
+      <!-- <link name="${prefix}vertex0"/>
       <link name="${prefix}vertex1"/>
       <link name="${prefix}vertex2"/>
@@ -461,5 +460,5 @@
         <parent link="${prefix}tabletop_link"/>
         <child link="${prefix}vertex4"/>
-      </joint>
+      </joint> -->
    </xacro:if>
   </xacro:macro>

Commit message: fix

File: battery_cell_description/urdf/battery_table.xacro (robot description, xacro)
@@ -268,5 +268,5 @@
     <child link="${prefix}tabletop_link"/>
   </joint>
-  <xacro:property name="battery_thickness" value="0.4" />
+  <xacro:property name="battery_thickness" value="0.005" />
   <xacro:property name="battery_width" value="${table_width}" />
   <xacro:property name="battery_length" value="${table_length}" />
