Commit message: completed moveit setup

File: battery_cell_moveit_config/config/gazebo_battery_cell.urdf (robot description, URDF)
Before this commit: robot battery_cell, 46 links, 45 joints
Links:
- added link omron_agv_base_link, mass 4000; collision mesh filename=file:///home/abel/projects/personal_ws/src/omron_agv_manipu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; visual mesh filename=file:///home/abel/projects/personal_ws/src/omron_agv_manipu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
- added link omron_arm_base_link
- added link omron_arm_flange
- added link omron_arm_link_0, mass 1.0; collision mesh filename=package://tm_description/meshes/tm12/collision/tm12-base_c.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; visual mesh filename=package://tm_description/meshes/tm12/visual/tm12-base.obj
- added link omron_arm_link_1, mass 7.6; collision mesh filename=package://tm_description/meshes/tm12/collision/tmr_750w_01_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; visual mesh filename=package://tm_description/meshes/tm12/visual/tmr_750w_01.obj
- added link omron_arm_link_2, mass 14.0239; collision mesh filename=package://tm_description/meshes/tm12/collision/tm12-arm1_c.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; visual mesh filename=package://tm_description/meshes/tm12/visual/tm12-arm1.obj
- added link omron_arm_link_3, mass 3.3577; collision mesh filename=package://tm_description/meshes/tm12/collision/tm12-arm2_c.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; visual mesh filename=package://tm_description/meshes/tm12/visual/tm12-arm2.obj
- added link omron_arm_link_4, mass 1.576; collision mesh filename=package://tm_description/meshes/tm5-900/collision/tmr_100w_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; visual mesh filename=package://tm_description/meshes/tm5-900/visual/tmr_100w_01.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
- added link omron_arm_link_5, mass 1.576; collision mesh filename=package://tm_description/meshes/tm5-900/collision/tmr_100w_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; visual mesh filename=package://tm_description/meshes/tm5-900/visual/tmr_100w_02.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
- added link omron_arm_link_6, mass 0.65; collision mesh filename=package://tm_description/meshes/tm5-900/collision/tmr_ee_c.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; visual mesh filename=package://tm_description/meshes/tm5-900/visual/tmr_ee.obj
- added link omron_base_link
- added link omron_base_x
- added link omron_base_y
- added link table_base_link
- added link table_leg1_link, mass 9.573825; collision box size=0.06 0.06 0.9; visual box size=0.06 0.06 0.9
- added link table_leg2_link, mass 9.573825; collision box size=0.06 0.06 0.9; visual box size=0.06 0.06 0.9
- added link table_leg3_link, mass 9.573825; collision box size=0.06 0.06 0.9; visual box size=0.06 0.06 0.9
- added link table_leg4_link, mass 9.573825; collision box size=0.06 0.06 0.9; visual box size=0.06 0.06 0.9
- added link table_tabletop_link, mass 9.573825; collision box size=1.5 1.48 0.015; visual box size=1.5 1.48 0.015
Joints:
- added joint omron_arm_base_fixed_joint: type fixed, parent omron_arm_base_link, child omron_arm_link_0, origin xyz=0.000000 0.000000 0.000000 rpy=0.000000 0.000000 0.000000
- added joint omron_arm_flange_fixed_joint: type fixed, parent omron_arm_link_6, child omron_arm_flange, origin xyz=0.000000 0.000000 0.000000 rpy=0.000000 0.000000 0.000000
- added joint omron_arm_joint_1: type revolute, parent omron_arm_link_0, child omron_arm_link_1, origin xyz=0.000000 0.000000 0.165200 rpy=0.000000 -0.000000 0.000000, axis 0 0 1, limit lower=-4.71238898038469 upper=4.71238898038469 effort=353 velocity=2.0943951023931953
- added joint omron_arm_joint_2: type revolute, parent omron_arm_link_1, child omron_arm_link_2, origin xyz=0.000000 0.000000 0.000000 rpy=-1.570796 -1.570796 0.000000, axis 0 0 1, limit lower=-3.141592653589793 upper=3.141592653589793 effort=353 velocity=2.0943951023931953
- added joint omron_arm_joint_3: type revolute, parent omron_arm_link_2, child omron_arm_link_3, origin xyz=0.636100 0.000000 0.000000 rpy=0.000000 -0.000000 0.000000, axis 0 0 1, limit lower=-2.897246558310587 upper=2.897246558310587 effort=157 velocity=3.141592653589793
- added joint omron_arm_joint_4: type revolute, parent omron_arm_link_3, child omron_arm_link_4, origin xyz=0.557900 0.000000 -0.156300 rpy=0.000000 -0.000000 1.570796, axis 0 0 1, limit lower=-3.141592653589793 upper=3.141592653589793 effort=54 velocity=3.141592653589793
- added joint omron_arm_joint_5: type revolute, parent omron_arm_link_4, child omron_arm_link_5, origin xyz=0.000000 -0.106000 0.000000 rpy=1.570796 -0.000000 0.000000, axis 0 0 1, limit lower=-3.141592653589793 upper=3.141592653589793 effort=54 velocity=3.141592653589793
- added joint omron_arm_joint_6: type revolute, parent omron_arm_link_5, child omron_arm_link_6, origin xyz=0.000000 -0.113150 0.000000 rpy=1.570796 -0.000000 0.000000, axis 0 0 1, limit lower=-4.71238898038469 upper=4.71238898038469 effort=54 velocity=3.141592653589793
- added joint omron_joint_rev: type revolute, parent omron_base_y, child omron_agv_base_link, origin xyz=0 0 0 rpy=0 0 0, axis 0 0 1, limit lower=-3.14159 upper=3.14159 effort=1000 velocity=3.14159
- added joint omron_joint_x: type prismatic, parent omron_base_link, child omron_base_x, origin xyz=0 0 0 rpy=0 0 0, axis 1 0 0, limit lower=-4.5 upper=0.5 effort=1000 velocity=2
- added joint omron_joint_y: type prismatic, parent omron_base_x, child omron_base_y, origin xyz=0 0 0 rpy=0 0 0, axis 0 1 0, limit lower=-1 upper=3 effort=1000 velocity=2
- added joint omron_lifter: type fixed, parent omron_agv_base_link, child omron_arm_base_link, origin xyz=0.2 -0.0 0.45 rpy= 0 0 0, axis 0 0 1
- added joint table_base_to_leg1: type fixed, parent table_base_link, child table_leg1_link, origin xyz=0.72 0.71 0 rpy=0 0 0
- added joint table_base_to_leg2: type fixed, parent table_base_link, child table_leg2_link, origin xyz=0.72 -0.71 0 rpy=0 0 0
- added joint table_base_to_leg3: type fixed, parent table_base_link, child table_leg3_link, origin xyz=-0.72 -0.71 0 rpy=0 0 0
- added joint table_base_to_leg4: type fixed, parent table_base_link, child table_leg4_link, origin xyz=-0.72 0.71 0 rpy=0 0 0
- added joint table_base_to_tabletop: type fixed, parent table_base_link, child table_tabletop_link, origin xyz=0 0 0.9 rpy=0 0 0
- added joint world_to_omron: type fixed, parent world, child omron_base_link, origin xyz=4.5 -3 0 rpy=0 0 0
- added joint world_to_table: type fixed, parent world, child table_base_link, origin xyz=1 -1 0 rpy=0 0 0
